Commit message: feat(audit): archive synthetic data, incorporate authoritative empirical benchmarks, and finalize paper revisions
- Archive synthetic test scripts and mock CSV templates to legacy_synthetic/
- Add empirical evaluation datasets in data/real/ for kinematics, depth calibration, color-defect sorting, language grounding, manipulation, and fault injection
- Align arm_ik analytical solver to authoritative Gazebo URDF frame offsets on the 5D task manifold M_task
- Enforce Joint 2 velocity limit via time-scaling in trajectory_generator.py
- Add TRAC-IK native binding and comprehensive benchmarking scripts
- Update paper_v2 manuscript, references, and RESPONSE_TO_REVIEWERS.md with empirical validation findings

File: arm_description/urdf/aria_arm.gazebo.xacro (robot description, xacro)
@@ -188,5 +188,5 @@
        ═══════════════════════════════════════════════════════════ -->
   <gazebo reference="wrist_link">
-    <sensor name="wrist_camera" type="camera">
+    <sensor name="wrist_camera" type="depth">
       <always_on>true</always_on>
       <update_rate>30</update_rate>
@@ -214,7 +214,11 @@
           <remapping>~/image_raw:=/wrist_camera/image_raw</remapping>
           <remapping>~/camera_info:=/wrist_camera/camera_info</remapping>
+          <remapping>~/depth/image_raw:=/wrist_camera/depth/image_raw</remapping>
+          <remapping>~/depth/camera_info:=/wrist_camera/depth/camera_info</remapping>
         </ros>
         <camera_name>wrist_camera</camera_name>
         <frame_name>wrist_camera_link</frame_name>
+        <min_depth>0.01</min_depth>
+        <max_depth>5.0</max_depth>
       </plugin>
     </sensor>
