Commit message: feat(u3): finalize infrastructure and launch configurations

File: arm_description/urdf/aria_arm.gazebo.xacro (robot description, xacro)
@@ -2,112 +2,70 @@
 <!-- ═══════════════════════════════════════════════════════════════
      ARIA Gazebo-Specific Configuration
-     Plugins, sensors, materials for Gazebo Harmonic (gz-sim)
+     Plugins, sensors, materials for Gazebo Classic 11
      Stage 1: CLEAN — all sensor noise set to zero
      ═══════════════════════════════════════════════════════════════ -->
 <robot xmlns:xacro="http://www.ros.org/wiki/xacro" name="aria_arm_gazebo">
   <!-- ═══════════════════════════════════════════════════════════
-       gz_ros2_control PLUGIN — bridges Gazebo ↔ ros2_control
-       Uses GazeboSimSystem for Gazebo Harmonic
+       gazebo_ros2_control PLUGIN — bridges Gazebo Classic ↔ ros2_control
+       Uses GazeboSystem for Gazebo Classic 11
        ═══════════════════════════════════════════════════════════ -->
   <gazebo>
-    <plugin filename="gz_ros2_control-system"
-            name="gz_ros2_control::GazeboSimROS2ControlPlugin">
+    <plugin filename="libgazebo_ros2_control.so"
+            name="gazebo_ros2_control">
       <parameters>$(find arm_control)/config/aria_controllers.yaml</parameters>
-      <ros>
-        <namespace>/</namespace>
-      </ros>
+      <robot_param>robot_description</robot_param>
+      <robot_param_node>robot_state_publisher</robot_param_node>
     </plugin>
   </gazebo>
   <!-- ═══════════════════════════════════════════════════════════
-       MATERIAL COLORS — Gazebo-specific (overrides URDF materials)
+       MATERIAL COLORS — Gazebo Classic specific
        ═══════════════════════════════════════════════════════════ -->
   <!-- Base: white -->
   <gazebo reference="base_link">
-    <material>
-      <ambient>0.95 0.95 0.95 1</ambient>
-      <diffuse>0.95 0.95 0.95 1</diffuse>
-      <specular>0.3 0.3 0.3 1</specular>
-    </material>
+    <material>Gazebo/White</material>
   </gazebo>
   <!-- Waist bracket: orange -->
   <gazebo reference="waist_link">
-    <material>
-      <ambient>0.95 0.55 0.10 1</ambient>
-      <diffuse>0.95 0.55 0.10 1</diffuse>
-      <specular>0.3 0.3 0.3 1</specular>
-    </material>
+    <material>Gazebo/Orange</material>
   </gazebo>
   <!-- Upper arm: orange -->
   <gazebo reference="upper_arm_link">
-    <material>
-      <ambient>0.95 0.55 0.10 1</ambient>
-      <diffuse>0.95 0.55 0.10 1</diffuse>
-      <specular>0.3 0.3 0.3 1</specular>
-    </material>
+    <material>Gazebo/Orange</material>
   </gazebo>
   <!-- Forearm: orange -->
   <gazebo reference="forearm_link">
-    <material>
-      <ambient>0.95 0.55 0.10 1</ambient>
-      <diffuse>0.95 0.55 0.10 1</diffuse>
-      <specular>0.3 0.3 0.3 1</specular>
-    </material>
+    <material>Gazebo/Orange</material>
   </gazebo>
   <!-- Wrist: orange -->
   <gazebo reference="wrist_link">
-    <material>
-      <ambient>0.95 0.55 0.10 1</ambient>
-      <diffuse>0.95 0.55 0.10 1</diffuse>
-      <specular>0.3 0.3 0.3 1</specular>
-    </material>
+    <material>Gazebo/Orange</material>
   </gazebo>
   <!-- Gripper holder: white -->
   <gazebo reference="gripper_holder_link">
-    <material>
-      <ambient>0.95 0.95 0.95 1</ambient>
-      <diffuse>0.95 0.95 0.95 1</diffuse>
-      <specular>0.3 0.3 0.3 1</specular>
-    </material>
+    <material>Gazebo/White</material>
   </gazebo>
   <!-- Gear housing: white -->
   <gazebo reference="gear_housing_link">
-    <material>
-      <ambient>0.95 0.95 0.95 1</ambient>
-      <diffuse>0.95 0.95 0.95 1</diffuse>
-      <specular>0.3 0.3 0.3 1</specular>
-    </material>
+    <material>Gazebo/White</material>
   </gazebo>
   <!-- Left finger pair: blue -->
   <gazebo reference="finger_left_1_link">
-    <material>
-      <ambient>0.20 0.40 0.85 1</ambient>
-      <diffuse>0.20 0.40 0.85 1</diffuse>
-      <specular>0.2 0.2 0.2 1</specular>
-    </material>
+    <material>Gazebo/Blue</material>
   </gazebo>
   <!-- Right finger pair: blue -->
   <gazebo reference="finger_right_1_link">
-    <material>
-      <ambient>0.20 0.40 0.85 1</ambient>
-      <diffuse>0.20 0.40 0.85 1</diffuse>
-      <specular>0.2 0.2 0.2 1</specular>
-    </material>
+    <material>Gazebo/Blue</material>
   </gazebo>
   <!-- Cameras: dark gray -->
   <gazebo reference="top_camera_link">
-    <material>
-      <ambient>0.25 0.25 0.25 1</ambient>
-      <diffuse>0.25 0.25 0.25 1</diffuse>
-    </material>
+    <material>Gazebo/DarkGrey</material>
   </gazebo>
   <gazebo reference="wrist_camera_link">
-    <material>
-      <ambient>0.25 0.25 0.25 1</ambient>
-      <diffuse>0.25 0.25 0.25 1</diffuse>
-    </material>
+    <material>Gazebo/DarkGrey</material>
   </gazebo>
   <!-- ═══════════════════════════════════════════════════════════
        TOP CAMERA SENSOR — Logitech C270
        1280×720, 60° HFOV, 30fps
+       Uses libgazebo_ros_camera.so for Gazebo Classic
        CLEAN: noise stddev = 0
        ═══════════════════════════════════════════════════════════ -->
@@ -133,5 +91,12 @@
         </noise>
       </camera>
-      <topic>top_camera/image_raw</topic>
+      <plugin name="top_camera_controller" filename="libgazebo_ros_camera.so">
+        <ros>
+          <remapping>~/image_raw:=/top_camera/image_raw</remapping>
+          <remapping>~/camera_info:=/top_camera/camera_info</remapping>
+        </ros>
+        <camera_name>top_camera</camera_name>
+        <frame_name>top_camera_link</frame_name>
+      </plugin>
     </sensor>
   </gazebo>
@@ -139,4 +104,5 @@
        WRIST CAMERA SENSOR — ESP32-CAM
        640×480, 66° HFOV, 15fps
+       Uses libgazebo_ros_camera.so for Gazebo Classic
        CLEAN: noise stddev = 0
        ═══════════════════════════════════════════════════════════ -->
@@ -162,5 +128,12 @@
         </noise>
       </camera>
-      <topic>wrist_camera/image_raw</topic>
+      <plugin name="wrist_camera_controller" filename="libgazebo_ros_camera.so">
+        <ros>
+          <remapping>~/image_raw:=/wrist_camera/image_raw</remapping>
+          <remapping>~/camera_info:=/wrist_camera/camera_info</remapping>
+        </ros>
+        <camera_name>wrist_camera</camera_name>
+        <frame_name>wrist_camera_link</frame_name>
+      </plugin>
     </sensor>
   </gazebo>
@@ -169,4 +142,5 @@
        6-axis: 3-axis gyro + 3-axis accelerometer
        100 Hz update rate
+       Uses libgazebo_ros_imu_sensor.so for Gazebo Classic
        CLEAN: all noise set to zero
        ═══════════════════════════════════════════════════════════ -->
@@ -177,45 +151,21 @@
       <imu>
         <angular_velocity>
-          <x>
-            <noise type="gaussian">
-              <mean>0.0</mean>
-              <stddev>0.0</stddev>  <!-- CLEAN -->
-            </noise>
-          </x>
-          <y>
-            <noise type="gaussian">
-              <mean>0.0</mean>
-              <stddev>0.0</stddev>  <!-- CLEAN -->
-            </noise>
-          </y>
-          <z>
-            <noise type="gaussian">
-              <mean>0.0</mean>
-              <stddev>0.0</stddev>  <!-- CLEAN -->
-            </noise>
-          </z>
+          <x><noise type="gaussian"><mean>0.0</mean><stddev>0.0</stddev></noise></x>
+          <y><noise type="gaussian"><mean>0.0</mean><stddev>0.0</stddev></noise></y>
+          <z><noise type="gaussian"><mean>0.0</mean><stddev>0.0</stddev></noise></z>
         </angular_velocity>
         <linear_acceleration>
-          <x>
-            <noise type="gaussian">
-              <mean>0.0</mean>
-              <stddev>0.0</stddev>  <!-- CLEAN -->
-            </noise>
-          </x>
-          <y>
-            <noise type="gaussian">
-              <mean>0.0</mean>
-              <stddev>0.0</stddev>  <!-- CLEAN -->
-            </noise>
-          </y>
-          <z>
-            <noise type="gaussian">
-              <mean>0.0</mean>
-              <stddev>0.0</stddev>  <!-- CLEAN -->
-            </noise>
-          </z>
+          <x><noise type="gaussian"><mean>0.0</mean><stddev>0.0</stddev></noise></x>
+          <y><noise type="gaussian"><mean>0.0</mean><stddev>0.0</stddev></noise></y>
+          <z><noise type="gaussian"><mean>0.0</mean><stddev>0.0</stddev></noise></z>
         </linear_acceleration>
       </imu>
-      <topic>mpu6050/imu_raw</topic>
+      <plugin name="imu_controller" filename="libgazebo_ros_imu_sensor.so">
+        <ros>
+          <remapping>~/out:=/mpu6050/imu_raw</remapping>
+        </ros>
+        <frame_name>imu_link</frame_name>
+        <initial_orientation_as_reference>false</initial_orientation_as_reference>
+      </plugin>
     </sensor>
   </gazebo>
@@ -223,5 +173,5 @@
        CONTACT SENSORS — on gripper fingers
        Detect objects grasped between finger pairs
-       Publishes to /gripper/contact
+       Uses libgazebo_ros_bumper.so for Gazebo Classic
        ═══════════════════════════════════════════════════════════ -->
   <gazebo reference="finger_left_1_link">
@@ -230,19 +180,16 @@
       <update_rate>30</update_rate>
       <contact>
-        <collision>finger_left_1_link_collision</collision>
+        <collision>finger_left_1_link_fixed_joint_lump__finger_left_1_link_collision_1</collision>
       </contact>
-      <topic>gripper/contact_left</topic>
+      <plugin name="contact_left_controller" filename="libgazebo_ros_bumper.so">
+        <ros>
+          <remapping>~/out:=/gripper/contact_left</remapping>
+        </ros>
+        <frame_name>finger_left_1_link</frame_name>
+      </plugin>
     </sensor>
     <!-- Finger surface friction -->
-    <collision>
-      <surface>
-        <friction>
-          <ode>
-            <mu>0.8</mu>
-            <mu2>0.8</mu2>
-          </ode>
-        </friction>
-      </surface>
-    </collision>
+    <mu1>0.8</mu1>
+    <mu2>0.8</mu2>
   </gazebo>
   <gazebo reference="finger_right_1_link">
@@ -251,19 +198,16 @@
       <update_rate>30</update_rate>
       <contact>
-        <collision>finger_right_1_link_collision</collision>
+        <collision>finger_right_1_link_fixed_joint_lump__finger_right_1_link_collision_1</collision>
       </contact>
-      <topic>gripper/contact_right</topic>
+      <plugin name="contact_right_controller" filename="libgazebo_ros_bumper.so">
+        <ros>
+          <remapping>~/out:=/gripper/contact_right</remapping>
+        </ros>
+        <frame_name>finger_right_1_link</frame_name>
+      </plugin>
     </sensor>
     <!-- Finger surface friction -->
-    <collision>
-      <surface>
-        <friction>
-          <ode>
-            <mu>0.8</mu>
-            <mu2>0.8</mu2>
-          </ode>
-        </friction>
-      </surface>
-    </collision>
+    <mu1>0.8</mu1>
+    <mu2>0.8</mu2>
   </gazebo>
   <!-- ═══════════════════════════════════════════════════════════

File: arm_description/urdf/aria_arm.urdf.xacro (robot description, xacro)
@@ -519,10 +519,10 @@
   <!-- ═══════════════════════════════════════════════════════════
        ROS2_CONTROL — Hardware Interface Configuration
-       In sim mode: gz_ros2_control/GazeboSimSystem (Gazebo handles physics)
-       In hardware mode: swap to arm_control/AriaHardwareInterface
-       ═══════════════════════════════════════════════════════════ -->
-  <ros2_control name="aria_arm_control" type="system">
+       Sim mode: gazebo_ros2_control/GazeboSystem (Gazebo Classic 11)
+       Hardware mode: swap to arm_control/AriaHardwareInterface
+       ═══════════════════════════════════════════════════════════ -->
+  <ros2_control name="GazeboSystem" type="system">
     <hardware>
-      <plugin>gz_ros2_control/GazeboSimSystem</plugin>
+      <plugin>gazebo_ros2_control/GazeboSystem</plugin>
     </hardware>
     <!-- Joint 1: Waist — MG995, Z-axis, -90° to +90° -->
@@ -580,4 +580,12 @@
       <state_interface name="velocity"/>
     </joint>
+    <!-- Mimic joint: Right finger pair mirrors gripper_joint -->
+    <joint name="finger_mimic_joint">
+      <param name="mimic">gripper_joint</param>
+      <param name="multiplier">-1</param>
+      <command_interface name="position"/>
+      <state_interface name="position"/>
+      <state_interface name="velocity"/>
+    </joint>
   </ros2_control>
 </robot>

Commit message: feat(sim): add tester workspace with multi-affordance benchmark objects, Jenga arena, multi-camera rig, and ARIA launcher

File: arm_description/urdf/aria_arm.gazebo.xacro (robot description, xacro)
@@ -64,53 +64,25 @@
     <material>Gazebo/DarkGrey</material>
   </gazebo>
-  <!-- ═══════════════════════════════════════════════════════════
-       TOP CAMERA SENSOR — Logitech C270
-       1280×720, 60° HFOV, 30fps
-       Uses libgazebo_ros_camera.so for Gazebo Classic
-       CLEAN: noise stddev = 0
-       ═══════════════════════════════════════════════════════════ -->
-  <gazebo reference="top_camera_link">
-    <sensor name="top_camera" type="camera">
-      <always_on>true</always_on>
-      <update_rate>30</update_rate>
-      <camera>
-        <horizontal_fov>1.0472</horizontal_fov>  <!-- 60 degrees -->
-        <image>
-          <width>1280</width>
-          <height>720</height>
-          <format>R8G8B8</format>
-        </image>
-        <clip>
-          <near>0.01</near>
-          <far>10.0</far>
-        </clip>
-        <noise>
-          <type>gaussian</type>
-          <mean>0.0</mean>
-          <stddev>0.0</stddev>  <!-- CLEAN: no noise in Stage 1 -->
-        </noise>
-      </camera>
-      <plugin name="top_camera_controller" filename="libgazebo_ros_camera.so">
-        <ros>
-          <remapping>~/image_raw:=/top_camera/image_raw</remapping>
-          <remapping>~/camera_info:=/top_camera/camera_info</remapping>
-        </ros>
-        <camera_name>top_camera</camera_name>
-        <frame_name>top_camera_link</frame_name>
-      </plugin>
-    </sensor>
-  </gazebo>
-  <!-- ═══════════════════════════════════════════════════════════
-       WRIST CAMERA SENSOR — ESP32-CAM
+  <!-- Preserve sensor joints from being lumped into parent link -->
+  <gazebo reference="wrist_camera_joint">
+    <preserveFixedJoint>true</preserveFixedJoint>
+  </gazebo>
+  <gazebo reference="imu_joint">
+    <preserveFixedJoint>true</preserveFixedJoint>
+  </gazebo>
+  <!-- ═══════════════════════════════════════════════════════════
+       WRIST CAMERA SENSOR — ESP32-CAM (attached to wrist_link)
        640×480, 66° HFOV, 15fps
        Uses libgazebo_ros_camera.so for Gazebo Classic
        CLEAN: noise stddev = 0
        ═══════════════════════════════════════════════════════════ -->
-  <gazebo reference="wrist_camera_link">
+  <gazebo reference="wrist_link">
     <sensor name="wrist_camera" type="camera">
       <always_on>true</always_on>
-      <update_rate>15</update_rate>
+      <update_rate>30</update_rate>
+      <visualize>false</visualize>
+      <pose>-0.02 0.055 0.0 0 0.52 1.5708</pose>
       <camera>
-        <horizontal_fov>1.1519</horizontal_fov>  <!-- 66 degrees -->
+        <horizontal_fov>1.35</horizontal_fov>  <!-- 77 degrees -->
         <image>
           <width>640</width>
