Commit message: feat(sim): add tester workspace with multi-affordance benchmark objects, Jenga arena, multi-camera rig, and ARIA launcher

File: arm_description/urdf/aria_arm.urdf.xacro (robot description, xacro)
@@ -1,311 +1,210 @@
 <?xml version="1.0"?>
 <!-- ═══════════════════════════════════════════════════════════════
-     ARIA 5-DoF Robotic Arm — URDF/Xacro Description
-     Techno-Tirupati kit with gear-driven gripper
-     Visual meshes from smart-methods/arduino-robot-arm repo
+     ARIA Robot Arm — URDF / Xacro Model
+     5-DOF Articulated Robotic Arm + 1-DOF Parallel Gripper
+     Actuator Limits: MG995 / MM995 (Waist, Shoulder, Elbow), SG90 (Wrist, Gripper)
+     Sensors: Wrist Camera (ESP32-CAM), MPU6050 6-Axis IMU
      ═══════════════════════════════════════════════════════════════ -->
 <robot xmlns:xacro="http://www.ros.org/wiki/xacro" name="aria_arm">
-  <!-- ═══ Include Gazebo-specific plugins ═══ -->
+  <!-- Include Gazebo-specific plugins and materials -->
   <xacro:include filename="$(find arm_description)/urdf/aria_arm.gazebo.xacro"/>
   <!-- ═══════════════════════════════════════════════════════════
-       DIMENSIONAL PARAMETERS — all from assembly manual
-       Units: meters, kilograms
-       ═══════════════════════════════════════════════════════════ -->
-  <!-- Base: white PLA cylinder (bottom housing) -->
-  <xacro:property name="base_radius"        value="0.040"/>  <!-- 80mm diameter -->
-  <xacro:property name="base_height"        value="0.070"/>  <!-- 70mm tall -->
-  <!-- Waist bracket: orange curved bracket on top of base -->
-  <xacro:property name="waist_width"        value="0.080"/>  <!-- 80mm wide -->
-  <xacro:property name="waist_depth"        value="0.040"/>  <!-- 40mm deep -->
-  <xacro:property name="waist_height"       value="0.035"/>  <!-- 35mm tall -->
-  <!-- Upper arm (Arm1): orange tube, slight curve, approximated as box -->
-  <xacro:property name="upper_arm_length"   value="0.145"/>  <!-- 145mm long -->
-  <xacro:property name="upper_arm_width"    value="0.025"/>  <!-- 25mm cross section -->
-  <xacro:property name="upper_arm_depth"    value="0.020"/>  <!-- 20mm cross section -->
-  <!-- Forearm (Arm2): orange rectangular housing -->
-  <xacro:property name="forearm_length"     value="0.115"/>  <!-- 115mm long -->
-  <xacro:property name="forearm_width"      value="0.030"/>  <!-- 30mm cross section -->
-  <xacro:property name="forearm_depth"      value="0.025"/>  <!-- 25mm cross section -->
-  <!-- Wrist (Arm3): small orange housing -->
-  <xacro:property name="wrist_length"       value="0.055"/>  <!-- 55mm long -->
-  <xacro:property name="wrist_width"        value="0.020"/>  <!-- 20mm cross section -->
-  <xacro:property name="wrist_depth"        value="0.018"/>  <!-- 18mm cross section -->
-  <!-- Gripper holder: white rectangular mount -->
-  <xacro:property name="gripper_holder_length" value="0.040"/>  <!-- 40mm long -->
-  <xacro:property name="gripper_holder_width"  value="0.025"/>  <!-- 25mm -->
-  <xacro:property name="gripper_holder_depth"  value="0.020"/>  <!-- 20mm -->
-  <!-- Gear housing: circular white gear mechanism -->
-  <xacro:property name="gear_radius"        value="0.015"/>  <!-- 30mm diameter -->
-  <xacro:property name="gear_height"        value="0.015"/>  <!-- 15mm tall -->
-  <!-- Fingers: curved blue plastic (each link = pair of 2 fingers) -->
-  <xacro:property name="finger_length"      value="0.080"/>  <!-- 80mm long -->
-  <xacro:property name="finger_width"       value="0.015"/>  <!-- 15mm wide -->
-  <xacro:property name="finger_depth"       value="0.005"/>  <!-- 5mm thick -->
-  <!-- Camera / sensor dimensions (small visual boxes) -->
-  <xacro:property name="camera_size"        value="0.025"/>  <!-- 25mm cube for camera visual -->
-  <!-- Mesh scale factor: STLs are in mm, convert to meters -->
-  <xacro:property name="mesh_scale"         value="0.001 0.001 0.001"/>
-  <!-- ═══════════════════════════════════════════════════════════
-       MASS PARAMETERS
-       PLA density = 1240 kg/m³
-       Includes servo mass at each joint location:
-         MG995 = 55g (waist, shoulder, elbow)
-         SG90  = 9g  (wrist_pitch, wrist_roll, gripper)
-       ═══════════════════════════════════════════════════════════ -->
-  <!-- base_link: PLA cylinder shell (~20g) + MG995 waist servo (55g) + hardware (75g) -->
-  <xacro:property name="base_mass"          value="0.150"/>
-  <!-- waist_link: PLA bracket (~45g) + MG995 shoulder servo (55g) -->
-  <xacro:property name="waist_mass"         value="0.100"/>
-  <!-- upper_arm_link: PLA tube (~65g) + MG995 elbow servo (55g) -->
-  <xacro:property name="upper_arm_mass"     value="0.120"/>
-  <!-- forearm_link: PLA housing (~55g) + SG90 wrist pitch servo (9g) + hardware (36g) -->
-  <xacro:property name="forearm_mass"       value="0.100"/>
-  <!-- wrist_link: PLA housing (~25g) + SG90 wrist roll servo (9g) -->
-  <xacro:property name="wrist_mass"         value="0.040"/>
-  <!-- gripper_holder_link: PLA mount (~15g) + SG90 gripper servo (9g) -->
-  <xacro:property name="gripper_holder_mass" value="0.025"/>
-  <!-- gear_housing_link: PLA gear housing (~20g) -->
-  <xacro:property name="gear_housing_mass"  value="0.020"/>
-  <!-- finger pair: PLA curved fingers (~10g per pair) -->
-  <xacro:property name="finger_mass"        value="0.010"/>
-  <!-- ═══════════════════════════════════════════════════════════
-       JOINT LIMITS (radians)
-       ═══════════════════════════════════════════════════════════ -->
-  <xacro:property name="waist_lower"        value="-1.5708"/>  <!-- -90° -->
-  <xacro:property name="waist_upper"        value="1.5708"/>   <!--  90° -->
-  <xacro:property name="shoulder_lower"     value="0.0"/>      <!--   0° -->
-  <xacro:property name="shoulder_upper"     value="3.1416"/>   <!-- 180° -->
-  <xacro:property name="elbow_lower"        value="0.0"/>      <!--   0° -->
-  <xacro:property name="elbow_upper"        value="2.6180"/>   <!-- 150° -->
-  <xacro:property name="wrist_pitch_lower"  value="-1.5708"/>  <!-- -90° -->
-  <xacro:property name="wrist_pitch_upper"  value="1.5708"/>   <!--  90° -->
-  <xacro:property name="wrist_roll_lower"   value="-1.5708"/>  <!-- -90° -->
-  <xacro:property name="wrist_roll_upper"   value="1.5708"/>   <!--  90° -->
-  <xacro:property name="gripper_lower"      value="0.0"/>      <!--   0° (closed) -->
-  <xacro:property name="gripper_upper"      value="0.7854"/>   <!--  45° (open)   -->
-  <!-- Joint velocity/effort limits (simulation values — higher than real servos for PID headroom) -->
-  <xacro:property name="mg995_effort"       value="10.0"/>     <!-- real: 1.0 Nm, sim needs headroom -->
-  <xacro:property name="mg995_velocity"     value="5.24"/>     <!-- ~300°/s max for MG995 -->
-  <xacro:property name="sg90_effort"        value="5.0"/>      <!-- real: 0.18 Nm, sim needs headroom -->
-  <xacro:property name="sg90_velocity"      value="10.47"/>    <!-- ~600°/s max for SG90 -->
-  <!-- ═══════════════════════════════════════════════════════════
-       MATERIAL DEFINITIONS (for RViz)
-       ═══════════════════════════════════════════════════════════ -->
-  <material name="white">
-    <color rgba="0.95 0.95 0.95 1.0"/>
-  </material>
-  <material name="orange">
-    <color rgba="0.95 0.55 0.10 1.0"/>
-  </material>
-  <material name="blue">
-    <color rgba="0.20 0.40 0.85 1.0"/>
-  </material>
-  <material name="dark_gray">
-    <color rgba="0.25 0.25 0.25 1.0"/>
-  </material>
-  <material name="light_gray">
-    <color rgba="0.75 0.75 0.75 1.0"/>
-  </material>
-  <!-- ═══════════════════════════════════════════════════════════
-       INERTIA MACROS — compute from box/cylinder formulas
-       ═══════════════════════════════════════════════════════════ -->
-  <!-- Solid box inertia: I = m/12 * (dim² sums)
-       x,y,z are full dimensions (not half) -->
-  <xacro:macro name="box_inertia" params="m x y z">
-    <inertial>
-      <mass value="${m}"/>
-      <inertia
-        ixx="${(1.0/12.0)*m*(y*y + z*z)}" ixy="0.0" ixz="0.0"
-        iyy="${(1.0/12.0)*m*(x*x + z*z)}" iyz="0.0"
-        izz="${(1.0/12.0)*m*(x*x + y*y)}"/>
-    </inertial>
-  </xacro:macro>
-  <!-- Solid cylinder inertia (axis along Z):
-       I_xx = I_yy = m/12*(3r² + h²), I_zz = m/2*r² -->
-  <xacro:macro name="cylinder_inertia" params="m r h">
-    <inertial>
-      <mass value="${m}"/>
-      <inertia
-        ixx="${(1.0/12.0)*m*(3.0*r*r + h*h)}" ixy="0.0" ixz="0.0"
-        iyy="${(1.0/12.0)*m*(3.0*r*r + h*h)}" iyz="0.0"
-        izz="${0.5*m*r*r}"/>
-    </inertial>
-  </xacro:macro>
-  <!-- ═══════════════════════════════════════════════════════════
-       WORLD FRAME — anchor point
+       PROPERTIES & LIMITS
+       ═══════════════════════════════════════════════════════════ -->
+  <xacro:property name="arm_mesh_scale"     value="0.00098 0.00098 0.00098"/>
+  <xacro:property name="gripper_mesh_scale" value="0.00098 0.00098 0.00098"/>
+  <!-- Joint Angle Limits (radians) -->
+  <xacro:property name="waist_lower"        value="-1.5708"/> <!-- -90 deg -->
+  <xacro:property name="waist_upper"        value="1.5708"/>  <!-- +90 deg -->
+  <xacro:property name="shoulder_lower"     value="-1.5708"/> <!-- -90 deg -->
+  <xacro:property name="shoulder_upper"     value="1.5708"/>  <!-- +90 deg -->
+  <xacro:property name="elbow_lower"        value="-1.5708"/> <!-- -90 deg -->
+  <xacro:property name="elbow_upper"        value="1.5708"/>  <!-- +90 deg -->
+  <xacro:property name="wrist_pitch_lower"  value="-1.5708"/> <!-- -90 deg -->
+  <xacro:property name="wrist_pitch_upper"  value="1.5708"/>  <!-- +90 deg -->
+  <xacro:property name="gripper_lower"      value="0.0"/>
+  <xacro:property name="gripper_upper"      value="1.047"/>   <!-- 60 deg open -->
+  <!-- Actuator Specifications (MG995 / MM995 & SG90 Servos) -->
+  <xacro:property name="mg995_effort"       value="25.0"/>
+  <xacro:property name="mg995_velocity"     value="3.5"/>
+  <xacro:property name="sg90_effort"        value="10.0"/>
+  <xacro:property name="sg90_velocity"      value="6.0"/>
+  <!-- ═══════════════════════════════════════════════════════════
+       MATERIALS (for RViz visualization)
+       ═══════════════════════════════════════════════════════════ -->
+  <material name="white"><color rgba="0.95 0.95 0.95 1.0"/></material>
+  <material name="orange"><color rgba="1.0 0.55 0.0 1.0"/></material>
+  <material name="blue"><color rgba="0.15 0.35 0.85 1.0"/></material>
+  <material name="dark_gray"><color rgba="0.25 0.25 0.25 1.0"/></material>
+  <!-- ═══════════════════════════════════════════════════════════
+       WORLD ANCHOR & FIXED TABLE ATTACHMENT
        ═══════════════════════════════════════════════════════════ -->
   <link name="world"/>
-  <!-- Fix base to table position: left-center of table, on surface -->
   <joint name="fixed_base" type="fixed">
     <parent link="world"/>
     <child link="base_link"/>
-    <origin xyz="-0.15 0.0 0.76" rpy="0 0 0"/>
-  </joint>
-  <!-- ═══════════════════════════════════════════════════════════
-       LINK 1: BASE — white PLA cylinder (bottom housing)
-       Contains MG995 servo for waist rotation
-       Visual: Base.stl from smart-methods/arduino-robot-arm
+    <origin xyz="0.0 0.0 0.614" rpy="0 0 1.5708"/>
+  </joint>
+  <!-- ═══════════════════════════════════════════════════════════
+       LINK 1: BASE — White cylindrical base housing
        ═══════════════════════════════════════════════════════════ -->
   <link name="base_link">
-    <visual>
+    <inertial>
+      <origin xyz="0 0 0.025" rpy="0 0 0"/>
+      <mass value="0.20"/>
+      <inertia ixx="0.001" ixy="0" ixz="0" iyy="0.001" iyz="0" izz="0.001"/>
+    </inertial>
+    <visual name="Base_Visual">
       <origin xyz="0 0 0" rpy="1.5708 0 0"/>
       <geometry>
-        <mesh filename="package://arm_description/meshes/stl/Base.stl" scale="${mesh_scale}"/>
+        <mesh filename="package://arm_description/meshes/stl/Base.stl" scale="${arm_mesh_scale}"/>
       </geometry>
       <material name="white"/>
     </visual>
-    <collision>
-      <origin xyz="0 0 ${base_height/2}" rpy="0 0 0"/>
-      <geometry>
-        <cylinder radius="${base_radius}" length="${base_height}"/>
-      </geometry>
-    </collision>
-    <!-- base_link: cylinder 80mm×70mm, mass≈150g (PLA shell + MG995 waist servo) -->
-    <xacro:cylinder_inertia m="${base_mass}" r="${base_radius}" h="${base_height}"/>
-  </link>
-  <!-- ═══════════════════════════════════════════════════════════
-       JOINT 1: WAIST — Z-axis rotation, MG995
-       At top of base cylinder
-       Damping increased for stability
+    <collision name="Base_Collision">
+      <origin xyz="-0.0029 0.00016 0.027" rpy="0 0 0"/>
+      <geometry>
+        <cylinder radius="0.0592" length="0.05469"/>
+      </geometry>
+    </collision>
+  </link>
+  <!-- ═══════════════════════════════════════════════════════════
+       JOINT 1: WAIST — MG995 / MM995 Servo
        ═══════════════════════════════════════════════════════════ -->
   <joint name="waist_joint" type="revolute">
+    <origin xyz="-0.00345 -1e-05 0.04449" rpy="0 0 0"/>
     <parent link="base_link"/>
     <child link="waist_link"/>
-    <origin xyz="0 0 ${base_height}" rpy="0 0 0"/>
-    <axis xyz="0 0 1"/>
-    <limit lower="${waist_lower}" upper="${waist_upper}"
-           effort="${mg995_effort}" velocity="${mg995_velocity}"/>
-    <dynamics damping="2.0" friction="0.3"/>
-  </joint>
-  <!-- ═══════════════════════════════════════════════════════════
-       LINK 2: WAIST BRACKET — orange curved bracket
-       Houses MG995 servo for shoulder rotation
-       Visual: Waist.stl from smart-methods/arduino-robot-arm
+    <axis xyz="0 0 1.0"/>
+    <limit lower="${waist_lower}" upper="${waist_upper}" effort="${mg995_effort}" velocity="${mg995_velocity}"/>
+    <dynamics damping="5.0" friction="0.5"/>
+  </joint>
+  <!-- ═══════════════════════════════════════════════════════════
+       LINK 2: WAIST — Orange waist bracket
        ═══════════════════════════════════════════════════════════ -->
   <link name="waist_link">
-    <visual>
+    <inertial>
+      <origin xyz="0 0 0.02" rpy="0 0 0"/>
+      <mass value="0.12"/>
+      <inertia ixx="0.001" ixy="0" ixz="0" iyy="0.001" iyz="0" izz="0.001"/>
+    </inertial>
+    <visual name="Waist_Visual">
       <origin xyz="0 0 0" rpy="1.5708 0 0"/>
       <geometry>
-        <mesh filename="package://arm_description/meshes/stl/Waist.stl" scale="${mesh_scale}"/>
+        <mesh filename="package://arm_description/meshes/stl/Waist.stl" scale="${arm_mesh_scale}"/>
       </geometry>
       <material name="orange"/>
     </visual>
-    <collision>
-      <origin xyz="0 0 ${waist_height/2}" rpy="0 0 0"/>
-      <geometry>
-        <box size="${waist_width} ${waist_depth} ${waist_height}"/>
-      </geometry>
-    </collision>
-    <!-- waist_link: box 80×40×35mm, mass≈100g (PLA bracket + MG995 shoulder servo) -->
-    <xacro:box_inertia m="${waist_mass}" x="${waist_width}" y="${waist_depth}" z="${waist_height}"/>
-  </link>
-  <!-- ═══════════════════════════════════════════════════════════
-       JOINT 2: SHOULDER — Y-axis rotation, MG995
-       At top of waist bracket
+    <collision name="Waist_Collision">
+      <origin xyz="0 0 0.02" rpy="0 0 0"/>
+      <geometry>
+        <box size="0.08 0.05 0.04"/>
+      </geometry>
+    </collision>
+  </link>
+  <!-- ═══════════════════════════════════════════════════════════
+       JOINT 2: SHOULDER — MG995 / MM995 Servo
        ═══════════════════════════════════════════════════════════ -->
   <joint name="shoulder_joint" type="revolute">
+    <origin xyz="0.00396 0.01369 0.03521" rpy="1.5708 0.03778 1.5708"/>
     <parent link="waist_link"/>
     <child link="upper_arm_link"/>
-    <origin xyz="0 0 ${waist_height}" rpy="0 0 0"/>
-    <axis xyz="0 1 0"/>
-    <limit lower="${shoulder_lower}" upper="${shoulder_upper}"
-           effort="${mg995_effort}" velocity="${mg995_velocity}"/>
-    <dynamics damping="3.0" friction="0.5"/>
-  </joint>
-  <!-- ═══════════════════════════════════════════════════════════
-       LINK 3: UPPER ARM (Arm1) — orange tube, 145mm
-       Slight curve, approximated as box for collision
-       Houses MG995 servo for elbow
-       Visual: Arm 01.stl from smart-methods/arduino-robot-arm
+    <axis xyz="0 0 1.0"/>
+    <limit lower="${shoulder_lower}" upper="${shoulder_upper}" effort="${mg995_effort}" velocity="${mg995_velocity}"/>
+    <dynamics damping="10.0" friction="1.0"/>
+  </joint>
+  <!-- ═══════════════════════════════════════════════════════════
+       LINK 3: UPPER ARM (Arm1) — Orange main link
        ═══════════════════════════════════════════════════════════ -->
   <link name="upper_arm_link">
-    <visual>
+    <inertial>
+      <origin xyz="0 0.06 0" rpy="0 0 0"/>
+      <mass value="0.15"/>
+      <inertia ixx="0.001" ixy="0" ixz="0" iyy="0.001" iyz="0" izz="0.001"/>
+    </inertial>
+    <visual name="Arm01_Visual">
       <origin xyz="0 0 0" rpy="0 0 0"/>
       <geometry>
-        <mesh filename="package://arm_description/meshes/stl/Arm 01.stl" scale="${mesh_scale}"/>
+        <mesh filename="package://arm_description/meshes/stl/Arm 01.stl" scale="${arm_mesh_scale}"/>
       </geometry>
       <material name="orange"/>
     </visual>
-    <collision>
-      <origin xyz="0 0 ${upper_arm_length/2}" rpy="0 0 0"/>
-      <geometry>
-        <box size="${upper_arm_width} ${upper_arm_depth} ${upper_arm_length}"/>
-      </geometry>
-    </collision>
-    <!-- upper_arm_link: box 25×20×145mm, mass≈120g (PLA tube + MG995 elbow servo) -->
-    <xacro:box_inertia m="${upper_arm_mass}" x="${upper_arm_width}" y="${upper_arm_depth}" z="${upper_arm_length}"/>
-  </link>
-  <!-- ═══════════════════════════════════════════════════════════
-       JOINT 3: ELBOW — Y-axis rotation, MG995
-       At junction of Arm1 and Arm2
+    <collision name="Arm01_Collision">
+      <origin xyz="-0.00032 0.05624 0.00439" rpy="0 0 0"/>
+      <geometry>
+        <box size="0.04221 0.16277 0.02051"/>
+      </geometry>
+    </collision>
+  </link>
+  <!-- ═══════════════════════════════════════════════════════════
+       JOINT 3: ELBOW — MG995 / MM995 Servo
        ═══════════════════════════════════════════════════════════ -->
   <joint name="elbow_joint" type="revolute">
+    <origin xyz="-7e-05 0.11689 -0.00792" rpy="-0.0013 -3.14159 0.03778"/>
     <parent link="upper_arm_link"/>
     <child link="forearm_link"/>
-    <origin xyz="0 0 ${upper_arm_length}" rpy="0 0 0"/>
-    <axis xyz="0 1 0"/>
-    <limit lower="${elbow_lower}" upper="${elbow_upper}"
-           effort="${mg995_effort}" velocity="${mg995_velocity}"/>
-    <dynamics damping="3.0" friction="0.5"/>
-  </joint>
-  <!-- ═══════════════════════════════════════════════════════════
-       LINK 4: FOREARM (Arm2) — orange rectangular housing, 115mm
-       Houses SG90 servo for wrist pitch
-       Visual: Arm 02.stl from smart-methods/arduino-robot-arm
+    <axis xyz="0 0 1.0"/>
+    <limit lower="${elbow_lower}" upper="${elbow_upper}" effort="${mg995_effort}" velocity="${mg995_velocity}"/>
+    <dynamics damping="8.0" friction="0.8"/>
+  </joint>
+  <!-- ═══════════════════════════════════════════════════════════
+       LINK 4: FOREARM (Arm2) — Orange forearm housing
        ═══════════════════════════════════════════════════════════ -->
   <link name="forearm_link">
-    <visual>
+    <inertial>
+      <origin xyz="0 0.06 0" rpy="0 0 0"/>
+      <mass value="0.10"/>
+      <inertia ixx="0.001" ixy="0" ixz="0" iyy="0.001" iyz="0" izz="0.001"/>
+    </inertial>
+    <visual name="Arm02_Visual">
       <origin xyz="0 0 0" rpy="-1.48894 -1.57209 1.57067"/>
       <geometry>
-        <mesh filename="package://arm_description/meshes/stl/Arm 02.stl" scale="${mesh_scale}"/>
+        <mesh filename="package://arm_description/meshes/stl/Arm 02.stl" scale="${arm_mesh_scale}"/>
       </geometry>
       <material name="orange"/>
     </visual>
-    <collision>
-      <origin xyz="0 0 ${forearm_length/2}" rpy="0 0 0"/>
-      <geometry>
-        <box size="${forearm_width} ${forearm_depth} ${forearm_length}"/>
-      </geometry>
-    </collision>
-    <!-- forearm_link: box 30×25×115mm, mass≈100g (PLA housing + SG90 wrist pitch servo) -->
-    <xacro:box_inertia m="${forearm_mass}" x="${forearm_width}" y="${forearm_depth}" z="${forearm_length}"/>
-  </link>
-  <!-- ═══════════════════════════════════════════════════════════
-       JOINT 4: WRIST PITCH — Y-axis rotation, SG90
-       At junction of Arm2 and Arm3
+    <collision name="Arm02_Collision">
+      <origin xyz="-0.00436 0.05688 0.00738" rpy="-1.48879 -1.57209 1.57066"/>
+      <geometry>
+        <box size="0.02681 0.16398 0.0384"/>
+      </geometry>
+    </collision>
+  </link>
+  <!-- ═══════════════════════════════════════════════════════════
+       JOINT 4: WRIST PITCH (wrist) — SG90 Micro Servo
        ═══════════════════════════════════════════════════════════ -->
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
Commit message: feat(vision): remove RealSense, restore Logitech C270 overhead camera and calibrate wrist camera optics

File: arm_description/urdf/aria_arm.gazebo.xacro (robot description, xacro)
@@ -82,5 +82,5 @@
       <update_rate>30</update_rate>
       <visualize>false</visualize>
-      <pose>-0.02 0.055 0.0 0 0.52 1.5708</pose>
+      <pose>-0.026 0.055 0.025 1.5708 0.0 -2.00</pose>
       <camera>
         <horizontal_fov>1.35</horizontal_fov>  <!-- 77 degrees -->

File: arm_description/urdf/aria_arm.urdf.xacro (robot description, xacro)
@@ -225,5 +225,5 @@
     <parent link="wrist_link"/>
     <child link="wrist_camera_link"/>
-    <origin xyz="-0.02 0.055 0.0" rpy="0 0.52 1.5708"/>
+    <origin xyz="-0.026 0.055 0.025" rpy="1.5708 0.0 -2.00"/>
   </joint>
   <link name="wrist_camera_link">

Commit message: Position wrist camera directly above and in middle of gripper claws pointing towards claws

File: arm_description/urdf/aria_arm.gazebo.xacro (robot description, xacro)
@@ -82,5 +82,5 @@
       <update_rate>30</update_rate>
       <visualize>false</visualize>
-      <pose>-0.026 0.055 0.025 1.5708 0.0 -2.00</pose>
+      <pose>0.025 0.050 -0.007 1.5708 0.0000 2.3036</pose>
       <camera>
         <horizontal_fov>1.35</horizontal_fov>  <!-- 77 degrees -->

File: arm_description/urdf/aria_arm.urdf.xacro (robot description, xacro)
@@ -225,5 +225,5 @@
     <parent link="wrist_link"/>
     <child link="wrist_camera_link"/>
-    <origin xyz="-0.026 0.055 0.025" rpy="1.5708 0.0 -2.00"/>
+    <origin xyz="0.025 0.050 -0.007" rpy="1.5708 0.0000 2.3036"/>
   </joint>
   <link name="wrist_camera_link">
