Commit message: Update gripper camera orientation and verify banana approach continuous frames

File: arm_description/urdf/aria_arm.gazebo.xacro (robot description, xacro)
@@ -82,5 +82,5 @@
       <update_rate>30</update_rate>
       <visualize>false</visualize>
-      <pose>0.025 0.050 -0.007 1.5708 0.0000 2.3036</pose>
+      <pose>0.025 0.050 -0.007 1.5708 0.0000 2.3358</pose>
       <camera>
         <horizontal_fov>1.35</horizontal_fov>  <!-- 77 degrees -->

File: arm_description/urdf/aria_arm.urdf.xacro (robot description, xacro)
@@ -225,5 +225,5 @@
     <parent link="wrist_link"/>
     <child link="wrist_camera_link"/>
-    <origin xyz="0.025 0.050 -0.007" rpy="1.5708 0.0000 2.3036"/>
+    <origin xyz="0.025 0.050 -0.007" rpy="1.5708 0.0000 2.3358"/>
   </joint>
   <link name="wrist_camera_link">

Commit message: Fix physics explosion, restore authentic 4-tier Jenga Tower, and stabilize object mass/contact parameters

File: arm_description/urdf/aria_arm.gazebo.xacro (robot description, xacro)
@@ -24,36 +24,71 @@
   <gazebo reference="base_link">
     <material>Gazebo/White</material>
+    <self_collide>false</self_collide>
+    <kp>100000.0</kp>
+    <kd>10.0</kd>
   </gazebo>
   <!-- Waist bracket: orange -->
   <gazebo reference="waist_link">
     <material>Gazebo/Orange</material>
+    <self_collide>false</self_collide>
+    <kp>100000.0</kp>
+    <kd>10.0</kd>
   </gazebo>
   <!-- Upper arm: orange -->
   <gazebo reference="upper_arm_link">
     <material>Gazebo/Orange</material>
+    <self_collide>false</self_collide>
+    <kp>100000.0</kp>
+    <kd>10.0</kd>
   </gazebo>
   <!-- Forearm: orange -->
   <gazebo reference="forearm_link">
     <material>Gazebo/Orange</material>
+    <self_collide>false</self_collide>
+    <kp>100000.0</kp>
+    <kd>10.0</kd>
   </gazebo>
   <!-- Wrist: orange -->
   <gazebo reference="wrist_link">
     <material>Gazebo/Orange</material>
+    <self_collide>false</self_collide>
+    <kp>100000.0</kp>
+    <kd>10.0</kd>
   </gazebo>
   <!-- Gripper holder: white -->
   <gazebo reference="gripper_holder_link">
     <material>Gazebo/White</material>
+    <self_collide>false</self_collide>
+    <kp>100000.0</kp>
+    <kd>10.0</kd>
   </gazebo>
   <!-- Gear housing: white -->
   <gazebo reference="gear_housing_link">
     <material>Gazebo/White</material>
+    <self_collide>false</self_collide>
+    <kp>100000.0</kp>
+    <kd>10.0</kd>
   </gazebo>
   <!-- Left finger pair: blue -->
   <gazebo reference="finger_left_1_link">
     <material>Gazebo/Blue</material>
+    <self_collide>false</self_collide>
+    <mu1>1.5</mu1>
+    <mu2>1.5</mu2>
+    <kp>50000.0</kp>
+    <kd>10.0</kd>
+    <minDepth>0.001</minDepth>
+    <maxVel>0.1</maxVel>
   </gazebo>
   <!-- Right finger pair: blue -->
   <gazebo reference="finger_right_1_link">
     <material>Gazebo/Blue</material>
+    <self_collide>false</self_collide>
+    <mu1>1.5</mu1>
+    <mu2>1.5</mu2>
+    <kp>50000.0</kp>
+    <kd>10.0</kd>
+    <minDepth>0.001</minDepth>
+    <maxVel>0.1</maxVel>
   </gazebo>
   <!-- Cameras: dark gray -->
@@ -82,5 +117,5 @@
       <update_rate>30</update_rate>
       <visualize>false</visualize>
-      <pose>0.025 0.050 -0.007 1.5708 0.0000 2.3358</pose>
+      <pose>0.015 0.040 -0.007 1.5708 0.2618 1.5708</pose>
       <camera>
         <horizontal_fov>1.35</horizontal_fov>  <!-- 77 degrees -->

File: arm_description/urdf/aria_arm.urdf.xacro (robot description, xacro)
@@ -225,5 +225,5 @@
     <parent link="wrist_link"/>
     <child link="wrist_camera_link"/>
-    <origin xyz="0.025 0.050 -0.007" rpy="1.5708 0.0000 2.3358"/>
+    <origin xyz="0.015 0.040 -0.007" rpy="1.5708 0.2618 1.5708"/>
   </joint>
   <link name="wrist_camera_link">

Commit message: feat(sim): stabilize physics, mesh collisions, and table safety envelope

File: arm_description/urdf/aria_arm.gazebo.xacro (robot description, xacro)
@@ -25,6 +25,8 @@
     <material>Gazebo/White</material>
     <self_collide>false</self_collide>
-    <kp>100000.0</kp>
-    <kd>10.0</kd>
+    <kp>50000.0</kp>
+    <kd>10.0</kd>
+    <minDepth>0.002</minDepth>
+    <maxVel>0.05</maxVel>
   </gazebo>
   <!-- Waist bracket: orange -->
@@ -32,6 +34,8 @@
     <material>Gazebo/Orange</material>
     <self_collide>false</self_collide>
-    <kp>100000.0</kp>
-    <kd>10.0</kd>
+    <kp>50000.0</kp>
+    <kd>10.0</kd>
+    <minDepth>0.002</minDepth>
+    <maxVel>0.05</maxVel>
   </gazebo>
   <!-- Upper arm: orange -->
@@ -39,6 +43,8 @@
     <material>Gazebo/Orange</material>
     <self_collide>false</self_collide>
-    <kp>100000.0</kp>
-    <kd>10.0</kd>
+    <kp>50000.0</kp>
+    <kd>10.0</kd>
+    <minDepth>0.002</minDepth>
+    <maxVel>0.05</maxVel>
   </gazebo>
   <!-- Forearm: orange -->
@@ -46,6 +52,8 @@
     <material>Gazebo/Orange</material>
     <self_collide>false</self_collide>
-    <kp>100000.0</kp>
-    <kd>10.0</kd>
+    <kp>50000.0</kp>
+    <kd>10.0</kd>
+    <minDepth>0.002</minDepth>
+    <maxVel>0.05</maxVel>
   </gazebo>
   <!-- Wrist: orange -->
@@ -53,6 +61,8 @@
     <material>Gazebo/Orange</material>
     <self_collide>false</self_collide>
-    <kp>100000.0</kp>
-    <kd>10.0</kd>
+    <kp>50000.0</kp>
+    <kd>10.0</kd>
+    <minDepth>0.002</minDepth>
+    <maxVel>0.05</maxVel>
   </gazebo>
   <!-- Gripper holder: white -->
@@ -60,6 +70,8 @@
     <material>Gazebo/White</material>
     <self_collide>false</self_collide>
-    <kp>100000.0</kp>
-    <kd>10.0</kd>
+    <kp>50000.0</kp>
+    <kd>10.0</kd>
+    <minDepth>0.002</minDepth>
+    <maxVel>0.05</maxVel>
   </gazebo>
   <!-- Gear housing: white -->
@@ -67,6 +79,8 @@
     <material>Gazebo/White</material>
     <self_collide>false</self_collide>
-    <kp>100000.0</kp>
-    <kd>10.0</kd>
+    <kp>50000.0</kp>
+    <kd>10.0</kd>
+    <minDepth>0.002</minDepth>
+    <maxVel>0.05</maxVel>
   </gazebo>
   <!-- Left finger pair: blue -->

File: arm_description/urdf/aria_arm.urdf.xacro (robot description, xacro)
@@ -52,6 +52,6 @@
     <inertial>
       <origin xyz="0 0 0.025" rpy="0 0 0"/>
-      <mass value="0.20"/>
-      <inertia ixx="0.001" ixy="0" ixz="0" iyy="0.001" iyz="0" izz="0.001"/>
+      <mass value="0.30"/>
+      <inertia ixx="0.0002" ixy="0" ixz="0" iyy="0.0002" iyz="0" izz="0.0003"/>
     </inertial>
     <visual name="Base_Visual">
@@ -78,5 +78,5 @@
     <axis xyz="0 0 1.0"/>
     <limit lower="${waist_lower}" upper="${waist_upper}" effort="${mg995_effort}" velocity="${mg995_velocity}"/>
-    <dynamics damping="5.0" friction="0.5"/>
+    <dynamics damping="0.1" friction="0.02"/>
   </joint>
   <!-- ═══════════════════════════════════════════════════════════
@@ -86,6 +86,6 @@
     <inertial>
       <origin xyz="0 0 0.02" rpy="0 0 0"/>
-      <mass value="0.12"/>
-      <inertia ixx="0.001" ixy="0" ixz="0" iyy="0.001" iyz="0" izz="0.001"/>
+      <mass value="0.20"/>
+      <inertia ixx="0.00015" ixy="0" ixz="0" iyy="0.00015" iyz="0" izz="0.0002"/>
     </inertial>
     <visual name="Waist_Visual">
@@ -112,5 +112,5 @@
     <axis xyz="0 0 1.0"/>
     <limit lower="${shoulder_lower}" upper="${shoulder_upper}" effort="${mg995_effort}" velocity="${mg995_velocity}"/>
-    <dynamics damping="10.0" friction="1.0"/>
+    <dynamics damping="0.1" friction="0.02"/>
   </joint>
   <!-- ═══════════════════════════════════════════════════════════
@@ -120,6 +120,6 @@
     <inertial>
       <origin xyz="0 0.06 0" rpy="0 0 0"/>
-      <mass value="0.15"/>
-      <inertia ixx="0.001" ixy="0" ixz="0" iyy="0.001" iyz="0" izz="0.001"/>
+      <mass value="0.18"/>
+      <inertia ixx="0.0002" ixy="0" ixz="0" iyy="0.00004" iyz="0" izz="0.0002"/>
     </inertial>
     <visual name="Arm01_Visual">
@@ -146,5 +146,5 @@
     <axis xyz="0 0 1.0"/>
     <limit lower="${elbow_lower}" upper="${elbow_upper}" effort="${mg995_effort}" velocity="${mg995_velocity}"/>
-    <dynamics damping="8.0" friction="0.8"/>
+    <dynamics damping="0.1" friction="0.02"/>
   </joint>
   <!-- ═══════════════════════════════════════════════════════════
@@ -154,6 +154,6 @@
     <inertial>
       <origin xyz="0 0.06 0" rpy="0 0 0"/>
-      <mass value="0.10"/>
-      <inertia ixx="0.001" ixy="0" ixz="0" iyy="0.001" iyz="0" izz="0.001"/>
+      <mass value="0.15"/>
+      <inertia ixx="0.00018" ixy="0" ixz="0" iyy="0.00003" iyz="0" izz="0.00018"/>
     </inertial>
     <visual name="Arm02_Visual">
@@ -180,5 +180,5 @@
     <axis xyz="0 0 1.0"/>
     <limit lower="${wrist_pitch_lower}" upper="${wrist_pitch_upper}" effort="${sg90_effort}" velocity="${sg90_velocity}"/>
-    <dynamics damping="4.0" friction="0.4"/>
+    <dynamics damping="0.05" friction="0.01"/>
   </joint>
   <!-- ═══════════════════════════════════════════════════════════
@@ -188,6 +188,6 @@
     <inertial>
       <origin xyz="0 0.02 0" rpy="0 0 0"/>
-      <mass value="0.05"/>
-      <inertia ixx="0.0005" ixy="0" ixz="0" iyy="0.0005" iyz="0" izz="0.0005"/>
+      <mass value="0.10"/>
+      <inertia ixx="0.00006" ixy="0" ixz="0" iyy="0.00006" iyz="0" izz="0.00006"/>
     </inertial>
     <visual name="Arm03_Visual">
@@ -206,19 +206,19 @@
   </link>
   <!-- ═══════════════════════════════════════════════════════════
-       IMU SENSOR LINK (MPU6050 mounted on wrist)
+       SENSOR LINK: MPU6050 6-Axis IMU (Inside wrist link)
        ═══════════════════════════════════════════════════════════ -->
   <joint name="imu_joint" type="fixed">
+    <origin xyz="0 0 0" rpy="0 0 0"/>
     <parent link="wrist_link"/>
     <child link="imu_link"/>
-    <origin xyz="0 0 0" rpy="0 0 0"/>
   </joint>
   <link name="imu_link">
     <inertial>
-      <mass value="0.002"/>
-      <inertia ixx="1e-8" ixy="0" ixz="0" iyy="1e-8" iyz="0" izz="1e-8"/>
-    </inertial>
-  </link>
-  <!-- ═══════════════════════════════════════════════════════════
-       WRIST CAMERA (ESP32-CAM mounted on wrist looking down at workspace)
+      <mass value="0.005"/>
+      <inertia ixx="1e-7" ixy="0" ixz="0" iyy="1e-7" iyz="0" izz="1e-7"/>
+    </inertial>
+  </link>
+  <!-- ═══════════════════════════════════════════════════════════
+       SENSOR LINK: WRIST CAMERA (In-Hand Gripper Vision)
        ═══════════════════════════════════════════════════════════ -->
   <joint name="wrist_camera_joint" type="fixed">
@@ -242,11 +242,11 @@
     <axis xyz="0 0 1.0"/>
     <limit lower="${gripper_lower}" upper="${gripper_upper}" effort="${sg90_effort}" velocity="${sg90_velocity}"/>
-    <dynamics damping="2.0" friction="0.2"/>
+    <dynamics damping="0.02" friction="0.005"/>
   </joint>
   <link name="finger_left_1_link">
     <inertial>
       <origin xyz="0 0 0.03" rpy="0 0 0"/>
-      <mass value="0.015"/>
-      <inertia ixx="0.0001" ixy="0" ixz="0" iyy="0.0001" iyz="0" izz="0.0001"/>
+      <mass value="0.03"/>
+      <inertia ixx="0.000015" ixy="0" ixz="0" iyy="0.000015" iyz="0" izz="0.000015"/>
     </inertial>
     <visual name="Gripper1_Visual">
@@ -258,7 +258,7 @@
     </visual>
     <collision name="Gripper1_Collision">
-      <origin xyz="0.00072 0.00044 0.03" rpy="-1.86728 0 0"/>
-      <geometry>
-        <box size="0.025 0.03 0.08"/>
+      <origin xyz="0 0 0" rpy="-1.86728 0 0"/>
+      <geometry>
+        <mesh filename="package://arm_description/meshes/stl/Gripper1.002.stl" scale="1.0 1.0 1.0"/>
       </geometry>
     </collision>
@@ -274,11 +274,11 @@
     <limit lower="${gripper_lower}" upper="${gripper_upper}" effort="${sg90_effort}" velocity="${sg90_velocity}"/>
     <mimic joint="gripper_joint" multiplier="1.0" offset="0.0"/>
-    <dynamics damping="2.0" friction="0.2"/>
+    <dynamics damping="0.02" friction="0.005"/>
   </joint>
   <link name="finger_right_1_link">
     <inertial>
       <origin xyz="0 0 0.03" rpy="0 0 0"/>
-      <mass value="0.015"/>
-      <inertia ixx="0.0001" ixy="0" ixz="0" iyy="0.0001" iyz="0" izz="0.0001"/>
+      <mass value="0.03"/>
+      <inertia ixx="0.000015" ixy="0" ixz="0" iyy="0.000015" iyz="0" izz="0.000015"/>
     </inertial>
     <visual name="Gripper2_Visual">
@@ -290,7 +290,7 @@
     </visual>
     <collision name="Gripper2_Collision">
-      <origin xyz="-0.00072 0.00044 0.03" rpy="-1.88476 0 0"/>
-      <geometry>
-        <box size="0.025 0.03 0.08"/>
+      <origin xyz="0 0 0" rpy="1.25673 0 0"/>
+      <geometry>
+        <mesh filename="package://arm_description/meshes/stl/Gripper2.stl" scale="1.0 1.0 1.0"/>
       </geometry>
     </collision>

Commit message: feat(sim): verified stable tabletop kinematics, implicit ODE joint dynamics, and display fix

File: arm_description/urdf/aria_arm.gazebo.xacro (robot description, xacro)
@@ -17,4 +17,32 @@
       <robot_param_node>robot_state_publisher</robot_param_node>
     </plugin>
+  </gazebo>
+  <!-- ═══════════════════════════════════════════════════════════
+       ROBUST JOINT DYNAMICS (Implicit Spring-Damper in ODE)
+       Prevents joint constraint explosion and shearing forces
+       ═══════════════════════════════════════════════════════════ -->
+  <gazebo reference="waist_joint">
+    <implicitSpringDamper>true</implicitSpringDamper>
+    <provideFeedback>true</provideFeedback>
+  </gazebo>
+  <gazebo reference="shoulder_joint">
+    <implicitSpringDamper>true</implicitSpringDamper>
+    <provideFeedback>true</provideFeedback>
+  </gazebo>
+  <gazebo reference="elbow_joint">
+    <implicitSpringDamper>true</implicitSpringDamper>
+    <provideFeedback>true</provideFeedback>
+  </gazebo>
+  <gazebo reference="wrist_pitch_joint">
+    <implicitSpringDamper>true</implicitSpringDamper>
+    <provideFeedback>true</provideFeedback>
+  </gazebo>
+  <gazebo reference="gripper_joint">
+    <implicitSpringDamper>true</implicitSpringDamper>
+    <provideFeedback>true</provideFeedback>
+  </gazebo>
+  <gazebo reference="finger_mimic_joint">
+    <implicitSpringDamper>true</implicitSpringDamper>
+    <provideFeedback>true</provideFeedback>
   </gazebo>
   <!-- ═══════════════════════════════════════════════════════════

File: arm_description/urdf/aria_arm.urdf.xacro (robot description, xacro)
@@ -258,7 +258,7 @@
     </visual>
     <collision name="Gripper1_Collision">
-      <origin xyz="0 0 0" rpy="-1.86728 0 0"/>
-      <geometry>
-        <mesh filename="package://arm_description/meshes/stl/Gripper1.002.stl" scale="1.0 1.0 1.0"/>
+      <origin xyz="0.005 0.020 0.035" rpy="-1.86728 0 0"/>
+      <geometry>
+        <box size="0.018 0.035 0.075"/>
       </geometry>
     </collision>
@@ -290,7 +290,7 @@
     </visual>
     <collision name="Gripper2_Collision">
-      <origin xyz="0 0 0" rpy="1.25673 0 0"/>
-      <geometry>
-        <mesh filename="package://arm_description/meshes/stl/Gripper2.stl" scale="1.0 1.0 1.0"/>
+      <origin xyz="-0.005 0.020 0.035" rpy="1.25673 0 0"/>
+      <geometry>
+        <box size="0.018 0.035 0.075"/>
       </geometry>
     </collision>

Commit message: feat(sim): add autonomous industrial manufacturing workcell with conveyor line, quality inspection, and finalized wrist camera angle
- Add aria_industrial_workcell.world with anchored, zero-tilt conveyor, photoelectric sensors, 4-slot assembly matrix, and defect reject bin
- Add Gazebo AriaConveyorPlugin for active belt motion, lateral centering, and queue spacing
- Add AriaGripperPlugin for reliable physical grasp and detach
- Finalize in-hand gripper camera pose from commit 58ffae390ee81e4d9a12573fffd9622512c7739e (0.025 0.050 -0.007 1.5708 0.0000 2.3358)
- Add SetConveyorPower service and industrial workcell autonomous sequencer and verification test suite
- Update CREDITS.md with open-source attributions

File: arm_description/urdf/aria_arm.gazebo.xacro (robot description, xacro)
@@ -19,4 +19,17 @@
   </gazebo>
   <!-- ═══════════════════════════════════════════════════════════
+       ARIA INDUSTRIAL GRIPPER PLUGIN — High-Fidelity Grasp & Release
+       ═══════════════════════════════════════════════════════════ -->
+  <gazebo>
+    <plugin filename="libaria_gripper_plugin.so"
+            name="aria_gripper_plugin">
+      <ros>
+        <namespace>/aria</namespace>
+      </ros>
+      <palm_link>wrist_link</palm_link>
+      <max_attach_dist>0.14</max_attach_dist>
+    </plugin>
+  </gazebo>
+  <!-- ═══════════════════════════════════════════════════════════
        ROBUST JOINT DYNAMICS (Implicit Spring-Damper in ODE)
        Prevents joint constraint explosion and shearing forces
@@ -116,10 +129,20 @@
     <material>Gazebo/Blue</material>
     <self_collide>false</self_collide>
-    <mu1>1.5</mu1>
-    <mu2>1.5</mu2>
-    <kp>50000.0</kp>
-    <kd>10.0</kd>
+    <mu1>2.5</mu1>
+    <mu2>2.5</mu2>
+    <kp>200000.0</kp>
+    <kd>20.0</kd>
     <minDepth>0.001</minDepth>
-    <maxVel>0.1</maxVel>
+    <maxVel>0.01</maxVel>
+    <torsional>
+      <ode>
+        <coefficient>10.0</coefficient>
+        <patch_radius>0.015</patch_radius>
+      </ode>
+    </torsional>
+    <bounce>
+      <restitution_coefficient>0.0</restitution_coefficient>
+      <threshold>1000000.0</threshold>
+    </bounce>
   </gazebo>
   <!-- Right finger pair: blue -->
@@ -127,10 +150,20 @@
     <material>Gazebo/Blue</material>
     <self_collide>false</self_collide>
-    <mu1>1.5</mu1>
-    <mu2>1.5</mu2>
-    <kp>50000.0</kp>
-    <kd>10.0</kd>
+    <mu1>2.5</mu1>
+    <mu2>2.5</mu2>
+    <kp>200000.0</kp>
+    <kd>20.0</kd>
     <minDepth>0.001</minDepth>
-    <maxVel>0.1</maxVel>
+    <maxVel>0.01</maxVel>
+    <torsional>
+      <ode>
+        <coefficient>10.0</coefficient>
+        <patch_radius>0.015</patch_radius>
+      </ode>
+    </torsional>
+    <bounce>
+      <restitution_coefficient>0.0</restitution_coefficient>
+      <threshold>1000000.0</threshold>
+    </bounce>
   </gazebo>
   <!-- Cameras: dark gray -->
@@ -159,5 +192,5 @@
       <update_rate>30</update_rate>
       <visualize>false</visualize>
-      <pose>0.015 0.040 -0.007 1.5708 0.2618 1.5708</pose>
+      <pose>0.025 0.050 -0.007 1.5708 0.0000 2.3358</pose>
       <camera>
         <horizontal_fov>1.35</horizontal_fov>  <!-- 77 degrees -->

File: arm_description/urdf/aria_arm.urdf.xacro (robot description, xacro)
@@ -225,5 +225,5 @@
     <parent link="wrist_link"/>
     <child link="wrist_camera_link"/>
-    <origin xyz="0.015 0.040 -0.007" rpy="1.5708 0.2618 1.5708"/>
+    <origin xyz="0.025 0.050 -0.007" rpy="1.5708 0.0000 2.3358"/>
   </joint>
   <link name="wrist_camera_link">
@@ -343,4 +343,11 @@
       <state_interface name="velocity"/>
     </joint>
+    <joint name="finger_mimic_joint">
+      <param name="mimic">gripper_joint</param>
+      <param name="multiplier">1</param>
+      <command_interface name="position"/>
+      <state_interface name="position"/>
+      <state_interface name="velocity"/>
+    </joint>
   </ros2_control>
 </robot>
