Commit message: fix(physics): align gripper collision pads, bind bumper sensors, and diagnose grasp slip

File: arm_description/urdf/aria_arm.gazebo.xacro (robot description, xacro)
@@ -126,4 +126,5 @@
   </gazebo>
   <!-- Left finger pair: blue -->
+  <!-- Left finger pair: blue -->
   <gazebo reference="finger_left_1_link">
     <material>Gazebo/Blue</material>
@@ -131,6 +132,6 @@
     <mu1>2.5</mu1>
     <mu2>2.5</mu2>
-    <kp>200000.0</kp>
-    <kd>20.0</kd>
+    <kp>1000000.0</kp>
+    <kd>50.0</kd>
     <minDepth>0.001</minDepth>
     <maxVel>0.01</maxVel>
@@ -145,4 +146,17 @@
       <threshold>1000000.0</threshold>
     </bounce>
+    <sensor name="gripper_contact_left" type="contact">
+      <always_on>true</always_on>
+      <update_rate>50</update_rate>
+      <contact>
+        <collision>finger_left_1_link_fixed_joint_lump__Gripper1_Collision_collision</collision>
+      </contact>
+      <plugin name="contact_left_controller" filename="libgazebo_ros_bumper.so">
+        <ros>
+          <remapping>bumper_states:=/gripper/contact_left</remapping>
+        </ros>
+        <frame_name>finger_left_1_link</frame_name>
+      </plugin>
+    </sensor>
   </gazebo>
   <!-- Right finger pair: blue -->
@@ -152,6 +166,6 @@
     <mu1>2.5</mu1>
     <mu2>2.5</mu2>
-    <kp>200000.0</kp>
-    <kd>20.0</kd>
+    <kp>1000000.0</kp>
+    <kd>50.0</kd>
     <minDepth>0.001</minDepth>
     <maxVel>0.01</maxVel>
@@ -166,4 +180,17 @@
       <threshold>1000000.0</threshold>
     </bounce>
+    <sensor name="gripper_contact_right" type="contact">
+      <always_on>true</always_on>
+      <update_rate>50</update_rate>
+      <contact>
+        <collision>finger_right_1_link_fixed_joint_lump__Gripper2_Collision_collision</collision>
+      </contact>
+      <plugin name="contact_right_controller" filename="libgazebo_ros_bumper.so">
+        <ros>
+          <remapping>bumper_states:=/gripper/contact_right</remapping>
+        </ros>
+        <frame_name>finger_right_1_link</frame_name>
+      </plugin>
+    </sensor>
   </gazebo>
   <!-- Cameras: dark gray -->
@@ -257,45 +284,4 @@
   </gazebo>
   <!-- ═══════════════════════════════════════════════════════════
-       CONTACT SENSORS — on gripper fingers
-       Detect objects grasped between finger pairs
-       Uses libgazebo_ros_bumper.so for Gazebo Classic
-       ═══════════════════════════════════════════════════════════ -->
-  <gazebo reference="finger_left_1_link">
-    <sensor name="gripper_contact_left" type="contact">
-      <always_on>true</always_on>
-      <update_rate>30</update_rate>
-      <contact>
-        <collision>finger_left_1_link_fixed_joint_lump__finger_left_1_link_collision_1</collision>
-      </contact>
-      <plugin name="contact_left_controller" filename="libgazebo_ros_bumper.so">
-        <ros>
-          <remapping>~/out:=/gripper/contact_left</remapping>
-        </ros>
-        <frame_name>finger_left_1_link</frame_name>
-      </plugin>
-    </sensor>
-    <!-- Finger surface friction -->
-    <mu1>0.8</mu1>
-    <mu2>0.8</mu2>
-  </gazebo>
-  <gazebo reference="finger_right_1_link">
-    <sensor name="gripper_contact_right" type="contact">
-      <always_on>true</always_on>
-      <update_rate>30</update_rate>
-      <contact>
-        <collision>finger_right_1_link_fixed_joint_lump__finger_right_1_link_collision_1</collision>
-      </contact>
-      <plugin name="contact_right_controller" filename="libgazebo_ros_bumper.so">
-        <ros>
-          <remapping>~/out:=/gripper/contact_right</remapping>
-        </ros>
-        <frame_name>finger_right_1_link</frame_name>
-      </plugin>
-    </sensor>
-    <!-- Finger surface friction -->
-    <mu1>0.8</mu1>
-    <mu2>0.8</mu2>
-  </gazebo>
-  <!-- ═══════════════════════════════════════════════════════════
        JOINT FRICTION — realistic but not overdone for Stage 1
        ═══════════════════════════════════════════════════════════ -->

File: arm_description/urdf/aria_arm.urdf.xacro (robot description, xacro)
@@ -258,7 +258,7 @@
     </visual>
     <collision name="Gripper1_Collision">
-      <origin xyz="0.005 0.020 0.035" rpy="-1.86728 0 0"/>
-      <geometry>
-        <box size="0.016 0.030 0.055"/>
+      <origin xyz="0.0012 0.045 -0.003" rpy="0 0 0"/>
+      <geometry>
+        <box size="0.024 0.075 0.018"/>
       </geometry>
     </collision>
@@ -290,7 +290,7 @@
     </visual>
     <collision name="Gripper2_Collision">
-      <origin xyz="-0.005 0.020 0.035" rpy="1.25673 0 0"/>
-      <geometry>
-        <box size="0.016 0.030 0.055"/>
+      <origin xyz="-0.0012 -0.045 0.001" rpy="0 0 0"/>
+      <geometry>
+        <box size="0.024 0.075 0.018"/>
       </geometry>
     </collision>

Commit message: fix(physics): prefix finger collision names with link name to enable Gazebo surface friction and bumper sensors

File: arm_description/urdf/aria_arm.gazebo.xacro (robot description, xacro)
@@ -150,5 +150,5 @@
       <update_rate>50</update_rate>
       <contact>
-        <collision>finger_left_1_link_fixed_joint_lump__Gripper1_Collision_collision</collision>
+        <collision>finger_left_1_link_collision_collision</collision>
       </contact>
       <plugin name="contact_left_controller" filename="libgazebo_ros_bumper.so">
@@ -184,5 +184,5 @@
       <update_rate>50</update_rate>
       <contact>
-        <collision>finger_right_1_link_fixed_joint_lump__Gripper2_Collision_collision</collision>
+        <collision>finger_right_1_link_collision_collision</collision>
       </contact>
       <plugin name="contact_right_controller" filename="libgazebo_ros_bumper.so">

File: arm_description/urdf/aria_arm.urdf.xacro (robot description, xacro)
@@ -257,5 +257,5 @@
       <material name="blue"/>
     </visual>
-    <collision name="Gripper1_Collision">
+    <collision name="finger_left_1_link_collision">
       <origin xyz="0.0012 0.045 -0.003" rpy="0 0 0"/>
       <geometry>
@@ -289,5 +289,5 @@
       <material name="blue"/>
     </visual>
-    <collision name="Gripper2_Collision">
+    <collision name="finger_right_1_link_collision">
       <origin xyz="-0.0012 -0.045 0.001" rpy="0 0 0"/>
       <geometry>

Commit message: feat(core): comprehensive autonomy stack upgrades, in-hand manipulation, MoveIt2 pipeline, and robust bringup
- Enhance arm agents with in-hand manipulation, Kalman tracking for moving targets, and truthful skill verification
- Add single-file master launch (aria.launch.py) and robust controller bring-up node (ensure_controllers.py)
- Finalize MoveIt2 configuration, setup assistant metadata, and controller launch pipelines
- Upgrade vision modules (SAM2, AprilTag calibration, Gaussian Splatting, 6D pose, transparent objects)
- Update VLA benchmarking, dataset export pipeline, training pipeline, and documentation

File: arm_description/urdf/aria_arm.gazebo.xacro (robot description, xacro)
@@ -107,23 +107,4 @@
     <maxVel>0.05</maxVel>
   </gazebo>
-  <!-- Gripper holder: white -->
-  <gazebo reference="gripper_holder_link">
-    <material>Gazebo/White</material>
-    <self_collide>false</self_collide>
-    <kp>50000.0</kp>
-    <kd>10.0</kd>
-    <minDepth>0.002</minDepth>
-    <maxVel>0.05</maxVel>
-  </gazebo>
-  <!-- Gear housing: white -->
-  <gazebo reference="gear_housing_link">
-    <material>Gazebo/White</material>
-    <self_collide>false</self_collide>
-    <kp>50000.0</kp>
-    <kd>10.0</kd>
-    <minDepth>0.002</minDepth>
-    <maxVel>0.05</maxVel>
-  </gazebo>
-  <!-- Left finger pair: blue -->
   <!-- Left finger pair: blue -->
   <gazebo reference="finger_left_1_link">
