Commit message: Save current working changes to test branch

File: arm_description/urdf/aria_arm.urdf.xacro (robot description, xacro)
@@ -2,6 +2,6 @@
 <!-- ═══════════════════════════════════════════════════════════════
      ARIA 5-DoF Robotic Arm — URDF/Xacro Description
-     Techno-Tirupati kit with NEW gear-driven gripper
-     Derived from assembly manual + photo measurements
+     Techno-Tirupati kit with gear-driven gripper
+     Visual meshes from smart-methods/arduino-robot-arm repo
      ═══════════════════════════════════════════════════════════════ -->
 <robot xmlns:xacro="http://www.ros.org/wiki/xacro" name="aria_arm">
@@ -44,4 +44,6 @@
   <!-- Camera / sensor dimensions (small visual boxes) -->
   <xacro:property name="camera_size"        value="0.025"/>  <!-- 25mm cube for camera visual -->
+  <!-- Mesh scale factor: STLs are in mm, convert to meters -->
+  <xacro:property name="mesh_scale"         value="0.001 0.001 0.001"/>
   <!-- ═══════════════════════════════════════════════════════════
        MASS PARAMETERS
@@ -82,8 +84,8 @@
   <xacro:property name="gripper_lower"      value="0.0"/>      <!--   0° (closed) -->
   <xacro:property name="gripper_upper"      value="0.7854"/>   <!--  45° (open)   -->
-  <!-- Joint velocity/effort limits -->
-  <xacro:property name="mg995_effort"       value="1.0"/>      <!-- ~1.0 Nm for MG995 -->
+  <!-- Joint velocity/effort limits (simulation values — higher than real servos for PID headroom) -->
+  <xacro:property name="mg995_effort"       value="10.0"/>     <!-- real: 1.0 Nm, sim needs headroom -->
   <xacro:property name="mg995_velocity"     value="5.24"/>     <!-- ~300°/s max for MG995 -->
-  <xacro:property name="sg90_effort"        value="0.18"/>     <!-- ~0.18 Nm for SG90 -->
+  <xacro:property name="sg90_effort"        value="5.0"/>      <!-- real: 0.18 Nm, sim needs headroom -->
   <xacro:property name="sg90_velocity"      value="10.47"/>    <!-- ~600°/s max for SG90 -->
   <!-- ═══════════════════════════════════════════════════════════
@@ -143,10 +145,11 @@
        LINK 1: BASE — white PLA cylinder (bottom housing)
        Contains MG995 servo for waist rotation
+       Visual: Base.stl from smart-methods/arduino-robot-arm
        ═══════════════════════════════════════════════════════════ -->
   <link name="base_link">
     <visual>
-      <origin xyz="0 0 ${base_height/2}" rpy="0 0 0"/>
-      <geometry>
-        <cylinder radius="${base_radius}" length="${base_height}"/>
+      <origin xyz="0 0 0" rpy="1.5708 0 0"/>
+      <geometry>
+        <mesh filename="package://arm_description/meshes/stl/Base.stl" scale="${mesh_scale}"/>
       </geometry>
       <material name="white"/>
@@ -164,4 +167,5 @@
        JOINT 1: WAIST — Z-axis rotation, MG995
        At top of base cylinder
+       Damping increased for stability
        ═══════════════════════════════════════════════════════════ -->
   <joint name="waist_joint" type="revolute">
@@ -172,15 +176,16 @@
     <limit lower="${waist_lower}" upper="${waist_upper}"
            effort="${mg995_effort}" velocity="${mg995_velocity}"/>
-    <dynamics damping="0.1" friction="0.05"/>
+    <dynamics damping="2.0" friction="0.3"/>
   </joint>
   <!-- ═══════════════════════════════════════════════════════════
        LINK 2: WAIST BRACKET — orange curved bracket
        Houses MG995 servo for shoulder rotation
+       Visual: Waist.stl from smart-methods/arduino-robot-arm
        ═══════════════════════════════════════════════════════════ -->
   <link name="waist_link">
     <visual>
-      <origin xyz="0 0 ${waist_height/2}" rpy="0 0 0"/>
-      <geometry>
-        <box size="${waist_width} ${waist_depth} ${waist_height}"/>
+      <origin xyz="0 0 0" rpy="1.5708 0 0"/>
+      <geometry>
+        <mesh filename="package://arm_description/meshes/stl/Waist.stl" scale="${mesh_scale}"/>
       </geometry>
       <material name="orange"/>
@@ -206,5 +211,5 @@
     <limit lower="${shoulder_lower}" upper="${shoulder_upper}"
            effort="${mg995_effort}" velocity="${mg995_velocity}"/>
-    <dynamics damping="0.1" friction="0.05"/>
+    <dynamics damping="3.0" friction="0.5"/>
   </joint>
   <!-- ═══════════════════════════════════════════════════════════
@@ -212,10 +217,11 @@
        Slight curve, approximated as box for collision
        Houses MG995 servo for elbow
+       Visual: Arm 01.stl from smart-methods/arduino-robot-arm
        ═══════════════════════════════════════════════════════════ -->
   <link name="upper_arm_link">
     <visual>
-      <origin xyz="0 0 ${upper_arm_length/2}" rpy="0 0 0"/>
-      <geometry>
-        <box size="${upper_arm_width} ${upper_arm_depth} ${upper_arm_length}"/>
+      <origin xyz="0 0 0" rpy="0 0 0"/>
+      <geometry>
+        <mesh filename="package://arm_description/meshes/stl/Arm 01.stl" scale="${mesh_scale}"/>
       </geometry>
       <material name="orange"/>
@@ -241,15 +247,16 @@
     <limit lower="${elbow_lower}" upper="${elbow_upper}"
            effort="${mg995_effort}" velocity="${mg995_velocity}"/>
-    <dynamics damping="0.1" friction="0.05"/>
+    <dynamics damping="3.0" friction="0.5"/>
   </joint>
   <!-- ═══════════════════════════════════════════════════════════
        LINK 4: FOREARM (Arm2) — orange rectangular housing, 115mm
        Houses SG90 servo for wrist pitch
+       Visual: Arm 02.stl from smart-methods/arduino-robot-arm
        ═══════════════════════════════════════════════════════════ -->
   <link name="forearm_link">
     <visual>
-      <origin xyz="0 0 ${forearm_length/2}" rpy="0 0 0"/>
-      <geometry>
-        <box size="${forearm_width} ${forearm_depth} ${forearm_length}"/>
+      <origin xyz="0 0 0" rpy="-1.48894 -1.57209 1.57067"/>
+      <geometry>
+        <mesh filename="package://arm_description/meshes/stl/Arm 02.stl" scale="${mesh_scale}"/>
       </geometry>
       <material name="orange"/>
@@ -275,15 +282,16 @@
     <limit lower="${wrist_pitch_lower}" upper="${wrist_pitch_upper}"
            effort="${sg90_effort}" velocity="${sg90_velocity}"/>
-    <dynamics damping="0.05" friction="0.02"/>
+    <dynamics damping="1.5" friction="0.3"/>
   </joint>
   <!-- ═══════════════════════════════════════════════════════════
        LINK 5: WRIST (Arm3) — small orange housing, 55mm
        Houses SG90 servo for wrist roll
+       Visual: Arm 03.stl from smart-methods/arduino-robot-arm
        ═══════════════════════════════════════════════════════════ -->
   <link name="wrist_link">
     <visual>
-      <origin xyz="0 0 ${wrist_length/2}" rpy="0 0 0"/>
-      <geometry>
-        <box size="${wrist_width} ${wrist_depth} ${wrist_length}"/>
+      <origin xyz="0 0 0" rpy="1.2416 1.55752 1.5708"/>
+      <geometry>
+        <mesh filename="package://arm_description/meshes/stl/Arm 03.stl" scale="${mesh_scale}"/>
       </geometry>
       <material name="orange"/>
@@ -331,15 +339,16 @@
     <limit lower="${wrist_roll_lower}" upper="${wrist_roll_upper}"
            effort="${sg90_effort}" velocity="${sg90_velocity}"/>
-    <dynamics damping="0.02" friction="0.01"/>
+    <dynamics damping="1.5" friction="0.3"/>
   </joint>
   <!-- ═══════════════════════════════════════════════════════════
        LINK 6: GRIPPER HOLDER — white rectangular mount, 40mm
        Houses SG90 gripper servo, mounts gear mechanism
+       Visual: Gripper1.stl from smart-methods/arduino-robot-arm
        ═══════════════════════════════════════════════════════════ -->
   <link name="gripper_holder_link">
     <visual>
-      <origin xyz="0 0 ${gripper_holder_length/2}" rpy="0 0 0"/>
-      <geometry>
-        <box size="${gripper_holder_width} ${gripper_holder_depth} ${gripper_holder_length}"/>
+      <origin xyz="0 0 0" rpy="0 0 0"/>
+      <geometry>
+        <mesh filename="package://arm_description/meshes/stl/Gripper1.stl" scale="1.0 1.0 1.0"/>
       </geometry>
       <material name="white"/>
@@ -379,4 +388,5 @@
        GEAR HOUSING — circular white gear mechanism
        Fixed to gripper holder, parent for finger joints
+       Visual: gear1.stl + gear2.stl from smart-methods/arduino-robot-arm
        ═══════════════════════════════════════════════════════════ -->
   <joint name="gear_housing_joint" type="fixed">
@@ -387,7 +397,7 @@
   <link name="gear_housing_link">
     <visual>
-      <origin xyz="0 0 ${gear_height/2}" rpy="0 0 0"/>
-      <geometry>
-        <cylinder radius="${gear_radius}" length="${gear_height}"/>
+      <origin xyz="0 0 0" rpy="0 0 0"/>
+      <geometry>
+        <mesh filename="package://arm_description/meshes/stl/gear1.stl" scale="1.0 1.0 1.0"/>
       </geometry>
       <material name="white"/>
@@ -414,15 +424,16 @@
     <limit lower="${gripper_lower}" upper="${gripper_upper}"
            effort="${sg90_effort}" velocity="${sg90_velocity}"/>
-    <dynamics damping="0.02" friction="0.01"/>
+    <dynamics damping="2.0" friction="0.3"/>
   </joint>
   <!-- ═══════════════════════════════════════════════════════════
        LEFT FINGER PAIR — 2 curved blue plastic fingers
        Driven directly by gripper_joint
+       Visual: Gripper1.002.stl from smart-methods/arduino-robot-arm
        ═══════════════════════════════════════════════════════════ -->
   <link name="finger_left_1_link">
     <visual>
-      <origin xyz="0 0 ${finger_length/2}" rpy="0 0 0"/>
-      <geometry>
-        <box size="${finger_width} ${finger_depth} ${finger_length}"/>
+      <origin xyz="0 0 0" rpy="-1.86728 0 0"/>
+      <geometry>
+        <mesh filename="package://arm_description/meshes/stl/Gripper1.002.stl" scale="1.0 1.0 1.0"/>
       </geometry>
       <material name="blue"/>
@@ -449,14 +460,15 @@
            effort="${sg90_effort}" velocity="${sg90_velocity}"/>
     <mimic joint="gripper_joint" multiplier="-1" offset="0"/>
-    <dynamics damping="0.02" friction="0.01"/>
+    <dynamics damping="0.1" friction="0.02"/>
   </joint>
   <!-- ═══════════════════════════════════════════════════════════
        RIGHT FINGER PAIR — 2 curved blue plastic fingers (mirrored)
+       Visual: Gripper2.stl from smart-methods/arduino-robot-arm
        ═══════════════════════════════════════════════════════════ -->
   <link name="finger_right_1_link">
     <visual>
-      <origin xyz="0 0 ${finger_length/2}" rpy="0 0 0"/>
-      <geometry>
-        <box size="${finger_width} ${finger_depth} ${finger_length}"/>
+      <origin xyz="0 0 0" rpy="1.25673 0 0"/>
+      <geometry>
+        <mesh filename="package://arm_description/meshes/stl/Gripper2.stl" scale="1.0 1.0 1.0"/>
       </geometry>
       <material name="blue"/>
@@ -489,12 +501,12 @@
   <!-- ═══════════════════════════════════════════════════════════
        TOP CAMERA — Logitech C270, fixed to world via stand
-       Position: 80cm above table, 40cm in front
-       Angle: 45° downward toward workspace
+       Position: top of camera stand pole (0.76m table + 0.80m pole)
+       Angle: 45° downward toward workspace center
        ═══════════════════════════════════════════════════════════ -->
   <joint name="top_camera_joint" type="fixed">
     <parent link="world"/>
     <child link="top_camera_link"/>
-    <!-- 40cm in front of origin, 80cm above table (table surface at 0.76m) -->
-    <origin xyz="0.40 0.0 0.80" rpy="0 0.7854 0"/>
+    <!-- Camera at top of stand pole, looking back at arm -->
+    <origin xyz="0.40 0.0 1.56" rpy="0 0.7854 3.14159"/>
   </joint>
   <link name="top_camera_link">
@@ -532,5 +544,7 @@
         <param name="max">${waist_upper}</param>
       </command_interface>
-      <state_interface name="position"/>
+      <state_interface name="position">
+        <param name="initial_value">0.0</param>
+      </state_interface>
       <state_interface name="velocity"/>
     </joint>
@@ -541,5 +555,7 @@
         <param name="max">${shoulder_upper}</param>
       </command_interface>
-      <state_interface name="position"/>
+      <state_interface name="position">
+        <param name="initial_value">1.5708</param>
+      </state_interface>
       <state_interface name="velocity"/>
     </joint>
@@ -550,5 +566,7 @@
         <param name="max">${elbow_upper}</param>
       </command_interface>
-      <state_interface name="position"/>
+      <state_interface name="position">
+        <param name="initial_value">1.3090</param>
+      </state_interface>
       <state_interface name="velocity"/>
     </joint>
@@ -559,5 +577,7 @@
         <param name="max">${wrist_pitch_upper}</param>
       </command_interface>
-      <state_interface name="position"/>
+      <state_interface name="position">
+        <param name="initial_value">0.0</param>
+      </state_interface>
       <state_interface name="velocity"/>
     </joint>
@@ -568,5 +588,7 @@
         <param name="max">${wrist_roll_upper}</param>
       </command_interface>
-      <state_interface name="position"/>
+      <state_interface name="position">
+        <param name="initial_value">0.0</param>
+      </state_interface>
       <state_interface name="velocity"/>
     </joint>
@@ -577,5 +599,7 @@
         <param name="max">${gripper_upper}</param>
       </command_interface>
-      <state_interface name="position"/>
+      <state_interface name="position">
+        <param name="initial_value">0.3491</param>
+      </state_interface>
       <state_interface name="velocity"/>
     </joint>

Commit message: fix(urdf): correct gripper mesh scaling and STL file references

File: arm_description/urdf/aria_arm.urdf.xacro (robot description, xacro)
@@ -126,5 +126,5 @@
       <origin xyz="0 0 0" rpy="0 0 0"/>
       <geometry>
-        <mesh filename="package://arm_description/meshes/stl/Arm 01.stl" scale="${arm_mesh_scale}"/>
+        <mesh filename="package://arm_description/meshes/stl/Arm_01.stl" scale="${arm_mesh_scale}"/>
       </geometry>
       <material name="orange"/>
@@ -160,5 +160,5 @@
       <origin xyz="0 0 0" rpy="-1.48894 -1.57209 1.57067"/>
       <geometry>
-        <mesh filename="package://arm_description/meshes/stl/Arm 02.stl" scale="${arm_mesh_scale}"/>
+        <mesh filename="package://arm_description/meshes/stl/Arm_02.stl" scale="${arm_mesh_scale}"/>
       </geometry>
       <material name="orange"/>
@@ -194,5 +194,5 @@
       <origin xyz="0 0 0" rpy="1.2416 1.55752 1.5708"/>
       <geometry>
-        <mesh filename="package://arm_description/meshes/stl/Arm 03.stl" scale="${arm_mesh_scale}"/>
+        <mesh filename="package://arm_description/meshes/stl/Arm_03.stl" scale="${arm_mesh_scale}"/>
       </geometry>
       <material name="orange"/>
@@ -253,5 +253,5 @@
       <origin xyz="0 0 0" rpy="-1.86728 0 0"/>
       <geometry>
-        <mesh filename="package://arm_description/meshes/stl/Gripper1.002.stl" scale="${gripper_mesh_scale}"/>
+        <mesh filename="package://arm_description/meshes/stl/Gripper1.002.stl" scale="1.0 1.0 1.0"/>
       </geometry>
       <material name="blue"/>
@@ -283,7 +283,7 @@
     </inertial>
     <visual name="Gripper2_Visual">
-      <origin xyz="0 0 0" rpy="-1.88476 0 0"/>
-      <geometry>
-        <mesh filename="package://arm_description/meshes/stl/Gripper1.003.stl" scale="${gripper_mesh_scale}"/>
+      <origin xyz="0 0 0" rpy="1.25673 0 0"/>
+      <geometry>
+        <mesh filename="package://arm_description/meshes/stl/Gripper2.stl" scale="1.0 1.0 1.0"/>
       </geometry>
       <material name="blue"/>

Commit message: Execute full 360 degree tabletop physical sweep demonstrating realistic multi-object contact dynamics

File: arm_description/urdf/aria_arm.urdf.xacro (robot description, xacro)
@@ -15,6 +15,6 @@
   <xacro:property name="gripper_mesh_scale" value="0.00098 0.00098 0.00098"/>
   <!-- Joint Angle Limits (radians) -->
-  <xacro:property name="waist_lower"        value="-1.5708"/> <!-- -90 deg -->
-  <xacro:property name="waist_upper"        value="1.5708"/>  <!-- +90 deg -->
+  <xacro:property name="waist_lower"        value="-3.14159"/> <!-- -180 deg -->
+  <xacro:property name="waist_upper"        value="3.14159"/>  <!-- +180 deg -->
   <xacro:property name="shoulder_lower"     value="-1.5708"/> <!-- -90 deg -->
   <xacro:property name="shoulder_upper"     value="1.5708"/>  <!-- +90 deg -->

Commit message: feat(sim): link joint clearances, natural object toppling, and grounded low-profile sweep

File: arm_description/urdf/aria_arm.urdf.xacro (robot description, xacro)
@@ -131,7 +131,7 @@
     </visual>
     <collision name="Arm01_Collision">
-      <origin xyz="-0.00032 0.05624 0.00439" rpy="0 0 0"/>
-      <geometry>
-        <box size="0.04221 0.16277 0.02051"/>
+      <origin xyz="-0.00032 0.058 0.00439" rpy="0 0 0"/>
+      <geometry>
+        <box size="0.038 0.082 0.020"/>
       </geometry>
     </collision>
@@ -165,7 +165,7 @@
     </visual>
     <collision name="Arm02_Collision">
-      <origin xyz="-0.00436 0.05688 0.00738" rpy="-1.48879 -1.57209 1.57066"/>
-      <geometry>
-        <box size="0.02681 0.16398 0.0384"/>
+      <origin xyz="-0.00436 0.062 0.00738" rpy="-1.48879 -1.57209 1.57066"/>
+      <geometry>
+        <box size="0.026 0.090 0.035"/>
       </geometry>
     </collision>
@@ -199,7 +199,7 @@
     </visual>
     <collision name="Arm03_Collision">
-      <origin xyz="-0.00062 0.00019 0.00049" rpy="1.24161 1.55752 1.5708"/>
-      <geometry>
-        <box size="0.035 0.06 0.025"/>
+      <origin xyz="-0.00062 0.015 0.00049" rpy="1.24161 1.55752 1.5708"/>
+      <geometry>
+        <box size="0.025 0.030 0.022"/>
       </geometry>
     </collision>
@@ -260,5 +260,5 @@
       <origin xyz="0.005 0.020 0.035" rpy="-1.86728 0 0"/>
       <geometry>
-        <box size="0.018 0.035 0.075"/>
+        <box size="0.016 0.030 0.055"/>
       </geometry>
     </collision>
@@ -292,5 +292,5 @@
       <origin xyz="-0.005 0.020 0.035" rpy="1.25673 0 0"/>
       <geometry>
-        <box size="0.018 0.035 0.075"/>
+        <box size="0.016 0.030 0.055"/>
       </geometry>
     </collision>

Commit message: fix(physics): align gripper collision pad orientations parallel to workpiece faces to eliminate wedge ejection force

File: arm_description/urdf/aria_arm.urdf.xacro (robot description, xacro)
@@ -258,5 +258,5 @@
     </visual>
     <collision name="finger_left_1_link_collision">
-      <origin xyz="0.0012 0.045 -0.003" rpy="0 0 0"/>
+      <origin xyz="0.0012 0.045 -0.003" rpy="-0.3054 0 0"/>
       <geometry>
         <box size="0.024 0.075 0.018"/>
@@ -290,5 +290,5 @@
     </visual>
     <collision name="finger_right_1_link_collision">
-      <origin xyz="-0.0012 -0.045 0.001" rpy="0 0 0"/>
+      <origin xyz="-0.0012 -0.045 0.001" rpy="-0.3054 0 0"/>
       <geometry>
         <box size="0.024 0.075 0.018"/>

Commit message: feat(audit): implement Phase 1 fixes A-J, freeze held-out prompt set, and prepare Phase 2 test suite

File: arm_description/urdf/aria_arm.urdf.xacro (robot description, xacro)
@@ -258,7 +258,7 @@
     </visual>
     <collision name="finger_left_1_link_collision">
-      <origin xyz="0.0012 0.045 -0.003" rpy="-0.3054 0 0"/>
-      <geometry>
-        <box size="0.024 0.075 0.018"/>
+      <origin xyz="0.0012 0.038 -0.003" rpy="-0.3054 0 0"/>
+      <geometry>
+        <box size="0.022 0.028 0.016"/>
       </geometry>
     </collision>
@@ -290,7 +290,7 @@
     </visual>
     <collision name="finger_right_1_link_collision">
-      <origin xyz="-0.0012 -0.045 0.001" rpy="-0.3054 0 0"/>
-      <geometry>
-        <box size="0.024 0.075 0.018"/>
+      <origin xyz="-0.0012 -0.038 0.001" rpy="-0.3054 0 0"/>
+      <geometry>
+        <box size="0.022 0.028 0.016"/>
       </geometry>
     </collision>

File: arm_ik/config/aria_arm.urdf (robot description, URDF)
Before this commit: robot aria_arm, 10 links, 9 joints
Links:
- link finger_left_1_link: geometry collision box size=0.022 0.028 0.016; visual mesh filename=package://arm_description/meshes/stl/Gripper1.002.stl scale=1.0 1.0 1.0
- link finger_right_1_link: geometry collision box size=0.022 0.028 0.016; visual mesh filename=package://arm_description/meshes/stl/Gripper2.stl scale=1.0 1.0 1.0

Commit message: fix(platform): reorient gripper pad collisions and reduce grip effort
The as-built pads were rotated 90 deg about the finger axis, so the pads
met the workpiece edge-on and splayed outward on contact.  Reorient both
pad collision boxes so their normals are exactly opposed at the grasp
opening (nL.d = +1.000, nR.(-d) = +1.000, nL.nR = -1.000 at g = 0.30),
shrink the boxes to 0.022 x 0.016 x 0.016 m, and drop gripper effort from
10 N.m to 0.18 N.m so the fingers cannot launch the 45 g cube.

This is a platform repair, recorded as a deviation from the frozen
as-built platform; P0/N1/N3/P0-WD results stand on the as-built platform
and N2 will run on the repaired platform under a new experiment ID.

File: arm_description/urdf/aria_arm.urdf.xacro (robot description, xacro)
@@ -33,4 +33,8 @@
   <xacro:property name="sg90_effort"        value="10.0"/>
   <xacro:property name="sg90_velocity"      value="6.0"/>
+  <!-- Gripper actuator limit: the SG90 stall torque is ~0.18 N*m, not 10 N*m.
+       The original 10 N*m limit produced 6 kN contact forces on a 40 mm cube. -->
+  <xacro:property name="gripper_effort"     value="0.18"/>
+  <xacro:property name="gripper_velocity"   value="6.0"/>
   <!-- ═══════════════════════════════════════════════════════════
        MATERIALS (for RViz visualization)
@@ -244,5 +248,5 @@
     <child link="finger_left_1_link"/>
     <axis xyz="0 0 1.0"/>
-    <limit lower="${gripper_lower}" upper="${gripper_upper}" effort="${sg90_effort}" velocity="${sg90_velocity}"/>
+    <limit lower="${gripper_lower}" upper="${gripper_upper}" effort="${gripper_effort}" velocity="${gripper_velocity}"/>
     <dynamics damping="0.02" friction="0.005"/>
   </joint>
@@ -261,7 +265,7 @@
     </visual>
     <collision name="finger_left_1_link_collision">
-      <origin xyz="0.0012 0.038 -0.003" rpy="-0.3054 0 0"/>
-      <geometry>
-        <box size="0.022 0.028 0.016"/>
+      <origin xyz="0.0012 0.038 -0.003" rpy="2.704300 -1.566512 0.0"/>
+      <geometry>
+        <box size="0.022 0.016 0.016"/>
       </geometry>
     </collision>
@@ -275,5 +279,5 @@
     <child link="finger_right_1_link"/>
     <axis xyz="0 0 1.0"/>
-    <limit lower="${gripper_lower}" upper="${gripper_upper}" effort="${sg90_effort}" velocity="${sg90_velocity}"/>
+    <limit lower="${gripper_lower}" upper="${gripper_upper}" effort="${gripper_effort}" velocity="${gripper_velocity}"/>
     <mimic joint="gripper_joint" multiplier="1.0" offset="0.0"/>
     <dynamics damping="0.02" friction="0.005"/>
@@ -293,7 +297,7 @@
     </visual>
     <collision name="finger_right_1_link_collision">
-      <origin xyz="-0.0012 -0.038 0.001" rpy="-0.3054 0 0"/>
-      <geometry>
-        <box size="0.022 0.028 0.016"/>
+      <origin xyz="-0.0012 -0.038 0.001" rpy="-2.678970 1.566213 0.0"/>
+      <geometry>
+        <box size="0.022 0.016 0.016"/>
       </geometry>
     </collision>
