Commit message: fix(platform): unpin workpieces, align gripper pads, document T1 blocker
- Gate the conveyor velocity override on belt motion: the plugin was
  zeroing each workpiece's vertical and angular velocity every tick while
  the belt was stopped, making a 50 mm pick physically impossible.
- Set pad friction through <gazebo reference> (mu=3) and re-orient the pad
  collision boxes so both faces are vertical and antiparallel at the grasp
  opening (measured dot -1.0000, tilt 0.00 deg).
- Enlarge the pad contact face from 10 mm to 30 mm.
- Add grasp bring-up/diagnostic tools under scripts/study/dev/.
- Record that the position-controlled jaws cannot regulate grip force, so
  T1 and P2-N2 remain not executable (DEVIATIONS D12, AUDIT 11.4).

File: arm_description/urdf/aria_arm.urdf.xacro (robot description, xacro)
@@ -265,7 +265,7 @@
     </visual>
     <collision name="finger_left_1_link_collision">
-      <origin xyz="0.0012 0.038 -0.003" rpy="2.704300 -1.566512 0.0"/>
-      <geometry>
-        <box size="0.022 0.016 0.016"/>
+      <origin xyz="0.0012 0.038 -0.003" rpy="-1.566536 0.309021 -2.005428"/>
+      <geometry>
+        <box size="0.030 0.016 0.016"/>
       </geometry>
     </collision>
@@ -297,7 +297,7 @@
     </visual>
     <collision name="finger_right_1_link_collision">
-      <origin xyz="-0.0012 -0.038 0.001" rpy="-2.678970 1.566213 0.0"/>
-      <geometry>
-        <box size="0.022 0.016 0.016"/>
+      <origin xyz="-0.0012 -0.038 0.001" rpy="-1.566715 -0.291439 1.116399"/>
+      <geometry>
+        <box size="0.030 0.016 0.016"/>
       </geometry>
     </collision>
@@ -364,3 +364,28 @@
     </joint>
   </ros2_control>
+  <!-- ═══════════════════════════════════════════════════════════
+       GAZEBO PAD CONTACT PROPERTIES
+       URDF has no <surface> element, so the pad friction and contact
+       stiffness must be set through Gazebo's own extension.  The default
+       (mu = 1.0, rigid kp) lets the jaws slide over a 40 mm cube: the cube
+       stays on the belt while the pads travel up past it.  These values
+       give the pads a high friction coefficient (mu = 3) and a controlled
+       contact stiffness.
+       ═══════════════════════════════════════════════════════════ -->
+  <gazebo reference="finger_left_1_link">
+    <mu1>3.0</mu1>
+    <mu2>3.0</mu2>
+    <kp>5000.0</kp>
+    <kd>50.0</kd>
+    <minDepth>0.002</minDepth>
+    <maxVel>0.005</maxVel>
+  </gazebo>
+  <gazebo reference="finger_right_1_link">
+    <mu1>3.0</mu1>
+    <mu2>3.0</mu2>
+    <kp>5000.0</kp>
+    <kd>50.0</kd>
+    <minDepth>0.002</minDepth>
+    <maxVel>0.005</maxVel>
+  </gazebo>
 </robot>
